File: rusefiSTI2004.kicad_sch (KiCad schematic)
At the start: 3 parts, among them M2 Module:mega-mcu100-f7/0.2, M3 Module-power_12and5V-0.3, M4 Module-output-0.3

Commit message: IGN,INJ AND ETB WIRED
wip WORKED ON IGNITION AND INJECTORS,etb
Parts:
- removed M2: Module:mega-mcu100-f7/0.2, AAmega-mcu100-f7:mega-mcu100-f7, symbol AAmega-mcu100:Module{colon}mega-mcu100-f7/0.2
- removed M3: Module-power_12and5V-0.3, AApower_12and5V:power_12and5V, symbol AApower_12and5V:Module-power_12and5V-0.3
- removed M4: Module-output-0.3, AAoutput:output, symbol AAoutput:Module-output-0.3
- added F1, F2, F3, F4, F5: nSMD005, hellen-one-common:PAD-1206-PAD, symbol hellen-one-common:Fuse-Pad-Pad
- added J1: 1-1376430-0, symbol rusefi_1-1376430-0_135pin:1-1376430-0
- added M1: Module-mega-mcu144-0.7, hellen-one-mega-mcu144-0.7:mega-mcu144, symbol hellen-one-mega-mcu144-0.7:Module-mega-mcu144-0.7
- added M13, M7: Module-knock-0.2, hellen-one-knock-0.2:knock, symbol hellen-one-knock-0.2:Module-knock-0.2
- added M14, M8: Module-power_12and5V-0.3, hellen-one-power_12and5V-0.3:power_12and5V, symbol hellen-one-power_12and5V-0.3:Module-power_12and5V-0.3
- added M2, M9: Module-motor-driver-0.1, hellen-one-motor-driver-0.1:motor-driver, symbol hellen-one-motor-driver-0.1:Module-motor-driver-0.1
- added M3: Module-wbo-0.5, hellen-one-wbo-0.5:wbo, symbol hellen-one-wbo-0.5:Module-wbo-0.5
- added M4: Module-can-0.1, hellen-one-can-0.1:can, symbol hellen-one-can-0.1:Module-can-0.1
- added M5, M6: Module-vr-discrete-0.5, hellen-one-vr-discrete-0.5:vr-discrete, symbol hellen-one-vr-discrete-0.5:Module-vr-discrete-0.5
- added R1: 33k, hellen-one-common:R0603, symbol hellen-one-common:Res
- added R2: 6.8k, hellen-one-common:R0603, symbol hellen-one-common:Res
Connections:
- new net: F1.1, J1.81
- new net: F5.1, J1.6
- new net: F2.1, J1.82
- new net: F3.1, J1.83
- new net: F4.1, J1.84
- new net +12V: M14.E2 (V12)
- new net +12V_BACK_UP: J1.85, M14.V1 (V12_PERM)
- new net +12V_ETB: F5.2, M2.N2 (12V_IN), M2.S1 (12V_IN)
- new net +12V_IGN: J1.15, M14.V2 (IN_VIGN)
- new net +12V_RAW: J1.71, J1.72, M14.V3 (V12_RAW), R1.1
- new net +3.3V: M1.N22 (V33), M1.N32 (V33), M2.W5 (3V3_IN)
- new net +3.3VA: M1.N28 (V33_SWITCHABLE)
- new net +5V: M14.E4 (V5)
- new net +5VA: M1.E38 (V5A_SWITCHABLE), M1.N30 (V5A_SWITCHABLE), M1.W2 (V5A_SWITCHABLE), M13.E1 (V5A), M5.E4 (V5_IN), M6.E4 (V5_IN)
- new net +5VAS: M14.V4 (5VP)
- new net APS_PS_5V: J1.46
- new net ETB_DIR: M1.N16 (IO1), M2.W2 (PWM)
- new net ETB_DIS: M1.N19 (IO2), M2.W4 (DIR)
- new net ETB_PWM: M1.E17 (OUT_PWM2), M2.W1 (DIS)
- new net FAN_RELAY_1: M1.E32 (OUT_INJ6)
- new net FAN_RELAY_2: M1.E33 (OUT_INJ7), M1.E34 (OUT_INJ8)
- new net FUEL_PUMP_SIGNAL1: J1.92
- new net FUEL_PUMP_SIGNAL2: J1.28
- new net GND: J1.1, J1.107, J1.108, J1.2, J1.3, J1.31, J1.62, J1.63, J1.64, J1.65, J1.66, J1.67, J1.70, J1.78, J1.97, M13.E2 (GND), M14.S1 (GND), M2.G (GND), M5.G (GND), M6.G (GND), R2.1
- new net GNDA: M1.E39 (GNDA), M1.W1 (GNDA)
- new net GND_INJECTORS: J1.7
- new net IGN: M1.N26 (IN_VIGN), M14.E3 (VIGN)
- new net INJ1: M1.E19 (OUT_INJ1)
- new net INJ2: M1.E18 (OUT_INJ2)
- new net INJ3: M1.E29 (OUT_INJ3)
- new net INJ4: M1.E30 (OUT_INJ4)
- new net IN_CAM_HALL_CAM_LH: J1.74
- new net IN_CAM_HALL_CAM_RH: J1.75
- new net IN_CLT: J1.102
- new net IN_CRANK: M1.S22 (IN_CRANK), M5.E3 (OUT), M6.E3 (OUT)
- new net IN_CRANK+: J1.76, M5.W2 (VR+), M6.W2 (VR+)
- new net IN_CRANK-: J1.22, J1.88, M5.W1 (VR-), M6.W1 (VR-)
- new net IN_ECT: J1.45, M1.S28 (IN_CLT)
- new net IN_FUEL_LEVEL: J1.51
- new net IN_IAT: J1.44, M1.S26 (IN_IAT)
- new net IN_KNOCK: M1.S23 (IN_KNOCK), M13.E3 (OUT_KNOCK)
- new net IN_KNOCK_RAW: J1.56, M13.W1 (IN_KNOCK)
- new net IN_MAP: J1.54, M1.S21 (IN_MAP1)
- new net IN_NEUTRAL_SWITCH: J1.9
- new net IN_PPS_MAIN: J1.48, M1.S31 (IN_PPS)
- new net IN_PPS_SUB: J1.59, M1.S33 (IN_PPS2)
- new net IN_PS_PRESSURE_SWIITCH: J1.10
- new net IN_STARTER_SWITCH: J1.8
- new net IN_TPS_MAIN: J1.49, M1.S30 (IN_TPS)
- new net IN_TPS_SUB: J1.60, M1.S32 (IN_TPS2)
- new net IN_TUMBLE_SENSOR_LH: J1.57
- new net IN_TUMBLE_SENSOR_RH: J1.58
- new net IN_VMAIN: M1.S10 (IN_AUX4), R1.2, R2.2
- new net IN_VSS: J1.93
- new net MAIN_RELAY: M1.E31 (OUT_INJ5)
- new net OUT_ELECTRONIC_THROTTE_RELAY: J1.101
- new net OUT_ETB+: J1.5, M2.S3 (OUT+)
- new net OUT_ETB-: J1.4, M2.S2 (OUT-)
- new net OUT_FAN_RELAY_1: J1.91
- new net OUT_FAN_RELAY_2: J1.90
- new net OUT_IGN1: F4.2, M1.W11 (IGN1), M1.W8 (IGN4), M1.W9 (IGN3)
- new net OUT_IGN2: F3.2, M1.W10 (IGN2)
- new net OUT_IGN3: F2.2
- new net OUT_IGN4: F1.2
- new net OUT_INJ1: J1.37
- new net OUT_INJ2: J1.36
- new net OUT_INJ3: J1.35
- new net OUT_INJ4: J1.34
- new net OUT_MAIN_RELAY: J1.17
- new net OUT_PURGE_CONTROL: J1.115
- new net OUT_TACH: J1.124
- new net OUT_VVT_LH+: J1.120
- new net OUT_VVT_LH-: J1.130
- new net OUT_VVT_RH+: J1.119
- new net OUT_VVT_RH-: J1.129
- new net OUT_WG: J1.133
- new net PG_5VP: M1.S3 (IN_D2), M14.E6 (PG_5VP)
- new net PWR_EN: M1.N29 (OUT_PWR_EN), M14.E5 (EN_5VP)
- new net SENSOR_PS_5V: J1.47
- new net THRESHOLD_VR_CR: M1.E26 (OUT_PWM6), M5.E1 (Thresh_IN), M6.E1 (Thresh_IN)
- new net VBAT: M1.N27 (VBAT), M14.E1 (VBAT)
- new net VREF: M1.S35 (VREF1), M13.W2 (VREF)
- new net VR_ANALOG_CR: M1.S18 (IN_RES3), M5.E2 (OUT_A), M6.E2 (OUT_A)
Other:
- added sheet INJ (INJ4.kicad_sch)
- added sheet LS1 (INJ4.kicad_sch)
- note added: "A: B134"
- note added: "B: B135"
- note added: "C: B136"
- note added: "D: B137"

Commit message: started laying it out
quick layout
Parts:
- J1: footprint (none) -> STI:1-1376430-0
Changed lines of the file:
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@@
 			)
 		)
-		(property "Footprint" ""
+		(property "Footprint" "STI:1-1376430-0"
 			(at 30.48 242.57 0)
 			(effects
@@
 		)
 		(property "Description" ""
+			(at 30.48 266.7 0)
+			(effects
+				(font
+					(size 1.27 1.27)
+				)
+				(hide yes)
+			)
+		)
+		(property "Manufacturer" ""
+			(at 30.48 266.7 0)
+			(effects
+				(font
+					(size 1.27 1.27)
+				)
+				(hide yes)
+			)
+		)
+		(property "Manufacturer Part Number" ""
+			(at 30.48 266.7 0)
+			(effects
+				(font
+					(size 1.27 1.27)
+				)
+				(hide yes)
+			)
+		)
+		(property "JLCPCB Part #" ""
 			(at 30.48 266.7 0)
 			(effects
@@
 			)
 		)
-		(property "Footprint" ""
+		(property "Footprint" "STI:1-1376430-0"
 			(at 30.48 340.36 0)
 			(effects
@@
 		)
 		(property "Description" ""
+			(at 30.48 364.49 0)
+			(effects
+				(font
+					(size 1.27 1.27)
+				)
+				(hide yes)
+			)
+		)
+		(property "Manufacturer" ""
+			(at 30.48 364.49 0)
+			(effects
+				(font
+					(size 1.27 1.27)
+				)
+				(hide yes)
+			)
+		)
+		(property "Manufacturer Part Number" ""
+			(at 30.48 364.49 0)
+			(effects
+				(font
+					(size 1.27 1.27)
+				)
+				(hide yes)
+			)
+		)
+		(property "JLCPCB Part #" ""
 			(at 30.48 364.49 0)
 			(effects
@@
 			)
 		)
-		(property "Footprint" ""
+		(property "Footprint" "STI:1-1376430-0"
 			(at 30.48 143.51 0)
 			(effects
@@
 		)
 		(property "Description" ""
+			(at 30.48 167.64 0)
+			(effects
+				(font
+					(size 1.27 1.27)
+				)
+				(hide yes)
+			)
+		)
+		(property "Manufacturer" ""
+			(at 30.48 167.64 0)
+			(effects
+				(font
+					(size 1.27 1.27)
+				)
+				(hide yes)
+			)
+		)
+		(property "Manufacturer Part Number" ""
+			(at 30.48 167.64 0)
+			(effects
+				(font
+					(size 1.27 1.27)
+				)
+				(hide yes)
+			)
+		)
+		(property "JLCPCB Part #" ""
 			(at 30.48 167.64 0)
 			(effects
@@
 			)
 		)
-		(property "Footprint" ""
+		(property "Footprint" "STI:1-1376430-0"
 			(at 27.94 40.64 0)
 			(effects
@@
 			(at 27.94 64.77 0)
 			(effects
+				(font
+					(size 1.27 1.27)
+				)
+				(hide yes)
+			)
+		)
+		(property "Manufacturer" ""
+			(at 27.94 64.77 0)
+			(effects
+				(font
+					(size 1.27 1.27)
+				)
+				(hide yes)
+			)
+		)
+		(property "Manufacturer Part Number" ""
+			(at 27.94 64.77 0)
+			(effects
+				(font
+					(size 1.27 1.27)
+				)
+				(hide yes)
+			)
+		)
+		(property "JLCPCB Part #" ""
+			(at 27.94 64.77 0)
+			(effects
