File: rusefiSTI2004.kicad_sch (KiCad schematic)
At the start: 19 parts, among them J1 1-1376430-0, M1 Module-mega-mcu144-0.7, M13 Module-knock-0.2, M14 Module-power_12and5V-0.3, M2 Module-motor-driver-0.1, M3 Module-wbo-0.5, M4 Module-can-0.1, M5 Module-vr-discrete-0.5, M6 Module-vr-discrete-0.5, M7 Module-knock-0.2, M8 Module-power_12and5V-0.3, M9 Module-motor-driver-0.1

Commit message: rev b: fix schematic wiring errors
- Ignition: MCU IGN3/IGN4 were labelled OUT_IGN1, shorting coils 1/3/4
  together and leaving coil 3/4 fuses undriven. Each IGN now goes to its own coil.
- ETB: labels at the motor driver were in PWM/DIR/DIS order but the module
  pins are DIS/PWM/DIR. OUT_PWM2 (timer) now drives PWM, IO1 -> DIR, IO2 -> DIS.
- OUT_INJ7 and OUT_INJ8 were both tied to FAN_RELAY_2. INJ8 is now free.
- Second VR module (M6) was paralleled on the crank. It now reads the LH cam
  (B8) into IN_CAM, with its own threshold (OUT_PWM3) and analog (IN_RES2);
  VR- goes to ground since the cam sensor is single-ended.
- Sensor 5V (APS C15, sensor C16) was floating. Both now fed from the
  protected +5VAS rail (M14 5VP).
- Vehicle speed (B27) now reaches M1 IN_VSS.

PCB still needs "Update PCB from Schematic" and re-routing in KiCad.

Co-Authored-By: Claude Opus 5.5 <noreply@anthropic.com>
Claude-Session: https://claude.ai/code/session_01Lq1NWipXY7ezEXP97C3qFj
Connections:
- net APS_PS_5V is gone; now on net +5VAS: J1.46
- net SENSOR_PS_5V is gone; now on net +5VAS: J1.47
- net ETB_DIR: now also M2.W4 (DIR); no longer M2.W2 (PWM)
- net ETB_DIS: now also M2.W1 (DIS); no longer M2.W4 (DIR)
- net ETB_PWM: now also M2.W2 (PWM); no longer M2.W1 (DIS)
- net FAN_RELAY_2: no longer M1.E34 (OUT_INJ8)
- net GND: now also M6.W1 (VR-)
- net IN_CAM_HALL_CAM_LH: now also M6.W2 (VR+)
- net IN_CRANK: no longer M6.E3 (OUT)
- net IN_CRANK+: no longer M6.W2 (VR+)
- net IN_CRANK-: no longer M6.W1 (VR-)
- net IN_VSS: now also M1.S25 (IN_VSS)
- net OUT_IGN1: no longer M1.W8 (IGN4), M1.W9 (IGN3)
- net OUT_IGN3: now also M1.W9 (IGN3)
- net OUT_IGN4: now also M1.W8 (IGN4)
- net THRESHOLD_VR_CR: no longer M6.E1 (Thresh_IN)
- net VR_ANALOG_CR: no longer M6.E2 (OUT_A)
- net THRESHOLD_VR_CAM: now reaches M1.E16 (OUT_PWM3)
- net THRESHOLD_VR_CAM: now also M6.E1 (Thresh_IN)
- net VR_ANALOG_CAM: now reaches M1.S14 (IN_RES2)
- net VR_ANALOG_CAM: now also M6.E2 (OUT_A)
- net IN_CAM: now reaches M1.S24 (IN_CAM)
- net IN_CAM: now also M6.E3 (OUT)
Changed lines of the file:
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@@
 	(wire
 		(pts
-			(xy 326.39 113.03) (xy 340.36 113.03)
-		)
-		(stroke
-			(width 0)
-			(type default)
-		)
-	)
-	(wire
-		(pts
 			(xy 241.3 52.07) (xy 259.08 52.07)
 		)
@@
 		)
 	)
-	(label "THRESHOLD_VR_CR"
+	(label "THRESHOLD_VR_CAM"
 		(at 265.43 196.85 180)
 		(fields_autoplaced yes)
@@
 		)
 	)
-	(label "FAN_RELAY_2"
-		(at 326.39 113.03 0)
-		(fields_autoplaced yes)
-		(effects
-			(font
-				(size 1.27 1.27)
-			)
-			(justify left bottom)
-		)
-	)
 	(label "INJ1"
 		(at 328.93 95.25 0)
@@
 		)
 	)
-	(label "IN_CRANK-"
-		(at 182.88 189.23 0)
-		(fields_autoplaced yes)
-		(effects
-			(font
-				(size 1.27 1.27)
-			)
-			(justify left bottom)
-		)
-	)
 	(label "VR_ANALOG_CR"
 		(at 265.43 162.56 180)
@@
 		)
 	)
-	(label "OUT_IGN1"
+	(label "OUT_IGN3"
 		(at 328.93 74.93 0)
 		(fields_autoplaced yes)
@@
 		)
 	)
-	(label "ETB_DIS"
+	(label "ETB_DIR"
 		(at 255.27 327.66 180)
 		(fields_autoplaced yes)
@@
 		)
 	)
-	(label "IN_CRANK+"
+	(label "IN_CAM_HALL_CAM_LH"
 		(at 182.88 186.69 0)
 		(fields_autoplaced yes)
@@
 		)
 	)
-	(label "VR_ANALOG_CR"
+	(label "VR_ANALOG_CAM"
 		(at 265.43 191.77 180)
 		(fields_autoplaced yes)
@@
 		)
 	)
-	(label "ETB_PWM"
+	(label "ETB_DIS"
 		(at 255.27 322.58 180)
 		(fields_autoplaced yes)
@@
 		)
 	)
-	(label "ETB_DIR"
+	(label "ETB_PWM"
 		(at 255.27 325.12 180)
 		(fields_autoplaced yes)
@@
 		)
 	)
-	(label "OUT_IGN1"
+	(label "OUT_IGN4"
 		(at 328.93 77.47 0)
 		(fields_autoplaced yes)
@@
 		)
 	)
-	(label "IN_CRANK"
+	(label "IN_CAM"
 		(at 265.43 186.69 180)
 		(fields_autoplaced yes)
@@
 		)
 	)
+	(symbol
+		(lib_id "power:GND")
+		(at 182.88 189.23 270)
+		(unit 1)
+		(exclude_from_sim no)
+		(in_bom yes)
+		(on_board yes)
+		(dnp no)
+		(property "Reference" "#PWR055"
+			(at 182.88 189.23 0)
+			(effects
+				(font
+					(size 1.27 1.27)
+				)
+				(hide yes)
+			)
+		)
+		(property "Value" "GND"
+			(at 182.88 189.23 0)
+			(effects
+				(font
+					(size 1.27 1.27)
+				)
+			)
+		)
+		(property "Footprint" ""
+			(at 182.88 189.23 0)
+			(effects
+				(font
+					(size 1.27 1.27)
+				)
+				(hide yes)
+			)
+		)
+		(property "Datasheet" ""
+			(at 182.88 189.23 0)
+			(effects
+				(font
+					(size 1.27 1.27)
+				)
+				(hide yes)
+			)
+		)
+		(property "Description" ""
+			(at 182.88 189.23 0)
+			(effects
+				(font
+					(size 1.27 1.27)
+				)
+				(hide yes)
+			)
+		)
+		(pin "1"
+		)
+		(instances
+			(project "rusefiSTI2004"
+				(path "/00d4d98c-a749-4bd2-a087-ea484becbbe4"
+					(reference "#PWR055")
+					(unit 1)
+				)
+			)
+		)
+	)
+	(label "IN_CAM"
+		(at 340.36 186.69 180)
+		(fields_autoplaced yes)
+		(effects
+			(font
+				(size 1.27 1.27)
+			)
+			(justify right bottom)
+		)
+	)
+	(label "VR_ANALOG_CAM"
+		(at 340.36 229.87 180)
+		(fields_autoplaced yes)
+		(effects
+			(font
+				(size 1.27 1.27)
+			)
+			(justify right bottom)
+		)
+	)
+	(label "THRESHOLD_VR_CAM"
+		(at 340.36 125.73 180)
+		(fields_autoplaced yes)
+		(effects
+			(font
+				(size 1.27 1.27)
+			)
+			(justify right bottom)
+		)
+	)
+	(symbol
+		(lib_id "alphax:+5VAS")
+		(at 49.53 160.02 90)
+		(unit 1)
+		(exclude_from_sim no)
+		(in_bom yes)
+		(on_board yes)
+		(dnp no)
+		(property "Reference" "#PWR056"
+			(at 49.53 160.02 0)
+			(effects
+				(font
+					(size 1.27 1.27)
+				)
+				(hide yes)
+			)
+		)
+		(property "Value" "+5VAS"
+			(at 49.53 160.02 0)
+			(effects
+				(font
+					(size 1.27 1.27)
+				)
+			)
+		)
+		(property "Footprint" ""
+			(at 49.53 160.02 0)
+			(effects
+				(font
+					(size 1.27 1.27)
+				)
+				(hide yes)
+			)
+		)
+		(property "Datasheet" ""
+			(at 49.53 160.02 0)
+			(effects
+				(font
+					(size 1.27 1.27)
+				)
+				(hide yes)
+			)
+		)
+		(property "Description" ""
+			(at 49.53 160.02 0)
+			(effects
+				(font
+					(size 1.27 1.27)
+				)
+				(hide yes)
+			)
+		)
+		(pin "1"
+		)
+		(instances
+			(project "rusefiSTI2004"
+				(path "/00d4d98c-a749-4bd2-a087-ea484becbbe4"
+					(reference "#PWR056")
+					(unit 1)
+				)
+			)
+		)
+	)
+	(symbol
+		(lib_id "alphax:+5VAS")
+		(at 49.53 162.56 90)
+		(unit 1)
+		(exclude_from_sim no)
+		(in_bom yes)
+		(on_board yes)
+		(dnp no)
+		(property "Reference" "#PWR057"
+			(at 49.53 162.56 0)
+			(effects
+				(font
+					(size 1.27 1.27)
+				)
+				(hide yes)
+			)
+		)
+		(property "Value" "+5VAS"
+			(at 49.53 162.56 0)
+			(effects
+				(font
+					(size 1.27 1.27)
+				)
+			)
+		)
+		(property "Footprint" ""
+			(at 49.53 162.56 0)
+			(effects
+				(font
+					(size 1.27 1.27)
+				)
+				(hide yes)
+			)
+		)
+		(property "Datasheet" ""
+			(at 49.53 162.56 0)
+			(effects
+				(font
+					(size 1.27 1.27)
+				)
+				(hide yes)
+			)
+		)
+		(property "Description" ""
+			(at 49.53 162.56 0)
+			(effects
+				(font
+					(size 1.27 1.27)
+				)
+				(hide yes)
+			)
+		)
+		(pin "1"
+		)
+		(instances
+			(project "rusefiSTI2004"
+				(path "/00d4d98c-a749-4bd2-a087-ea484becbbe4"
+					(reference "#PWR057")
+					(unit 1)
+				)
+			)
+		)
+	)
+	(label "IN_VSS"
+		(at 340.36 189.23 180)
+		(fields_autoplaced yes)
+		(effects
+			(font
+				(size 1.27 1.27)
+			)
+			(justify right bottom)
+		)
+	)

Commit message: Rev b wiring: fix pinout errors, wire the car's needed signals
Wrong before (from the FSM cross-check):
- MAF/MAP swapped: C23 -> IN_MAF (IN_SENS1), C22 -> IN_MAP (IN_MAP1)
- D7 injector ground floating -> GND; A34 -> GND; stray D22 removed from IN_CRANK-
- A1 clutch was IN_CLT (rusEFI coolant) -> IN_CLUTCH

Cams are 3-wire Hall (WI-114), not VR: M6 off the LH cam; B8 -> IN_CAM, B9 -> IN_AUX1.

Newly wired: neutral/PS (IN_AUX2/3), starter, A/C request, brake 1/2, clutch on 340k inputs with 4.7k pull-downs (R19-R23); TGV pots (IN_MAP2/3); fuel level (IN_AT1); rear O2 (IN_O2S); FPCU command B26 <- IGN5 (5 V PWM).
Two more INJ4 low-side sheets (LS2/LS3, Q9-Q16): wastegate, AVCS RH/LH (-) on OUT_PWM1/4/5, purge, MIL, rear O2 heater, A/C relay, tach. AVCS (+) A18/A19 to +12V_RAW (main relay).
TGV motors on M9 (both banks in parallel): OUT_IO12/IO3/IO4.

Verified: every new net's members checked against the plan in the kicad-cli netlist; ERC errors 308 -> 235, no new error types; tools/pinout_check.py: 47 -> 78 OK. Pin map in documents/README.md. PCB not yet updated from the schematic.

Co-Authored-By: Claude Opus 5.5 <noreply@anthropic.com>
Parts:
- added R19, R20, R21, R22, R23: 4.7k, hellen-one-common:R0603, symbol hellen-one-common:Res
Connections:
- net GND_INJECTORS is gone; now on net GND: J1.7
- net IN_CAM_HALL_CAM_RH is gone; now on net IN_CAM_RH: J1.75
- net IN_CLT is gone; now on net IN_CLUTCH: J1.102
- net IN_PS_PRESSURE_SWIITCH is gone; now on net IN_PS_PRESSURE_SWITCH: J1.10
- net OUT_VVT_LH+ is gone; now on net +12V_RAW: J1.120
- net OUT_VVT_RH+ is gone; now on net +12V_RAW: J1.119
- net +12V_RAW: now also M9.N2 (12V_IN), M9.S1 (12V_IN)
- net +3.3V: now also M9.W5 (3V3_IN)
- net FUEL_PUMP_SIGNAL1: now also M1.W7 (IGN5)
- net GND: now also J1.135, M9.G (GND), R19.2, R20.2, R21.2, R22.2, R23.2
- net IN_CAM: now also J1.74; no longer M6.E3 (OUT)
- net IN_CRANK-: no longer J1.22
- net IN_FUEL_LEVEL: now also M1.S27 (IN_AT1)
- net IN_MAP: now also J1.53; no longer J1.54
- net IN_NEUTRAL_SWITCH: now also M1.S12 (IN_AUX2)
- net IN_STARTER_SWITCH: now also M1.S8 (IN_SENS2), R19.1
- net IN_TUMBLE_SENSOR_LH: now also M1.S20 (IN_MAP2)
- net IN_TUMBLE_SENSOR_RH: now also M1.S19 (IN_MAP3)
- net O2_HEATER_REAR: now reaches M1.E12 (OUT_IO2)
- net TGV_PWM: now reaches M1.E13 (OUT_IO12)
- net TGV_PWM: now also M9.W2 (PWM)
- net VVT_LH: now reaches M1.E14 (OUT_PWM5)
- net VVT_RH: now reaches M1.E15 (OUT_PWM4)
- net TACH: now reaches M1.E21 (OUT_IO4)
- net PURGE: now reaches M1.E25 (OUT_PWM7)
- net WG: now reaches M1.E27 (OUT_PWM1)
- net AC_RELAY: now reaches M1.E6 (OUT_IO3)
- net MIL: now reaches M1.E8 (OUT_IO1)
- net TGV_DIS: now reaches M1.N20 (IO4)
- net TGV_DIS: now also M9.W1 (DIS)
- net TGV_DIR: now reaches M1.N21 (IO3)
- net TGV_DIR: now also M9.W4 (DIR)
- net IN_PS_PRESSURE_SWITCH: now reaches M1.S11 (IN_AUX3)
- net IN_CAM_RH: now reaches M1.S13 (IN_AUX1)
- net IN_BRAKE_SW1: now reaches M1.S15 (IN_O2S2)
- net IN_BRAKE_SW1: now also J1.40, R23.1
- net IN_O2S: now reaches M1.S16 (IN_O2S)
- net IN_O2S: now also J1.25
- net IN_CLUTCH: now reaches M1.S17 (IN_RES1)
- net IN_CLUTCH: now also R22.1
- net IN_BRAKE_SW2: now reaches M1.S6 (IN_SENS4)
- net IN_BRAKE_SW2: now also J1.39, R21.1
- net IN_AC_REQUEST: now reaches M1.S7 (IN_SENS3)
- net IN_AC_REQUEST: now also J1.16, R20.1
- net IN_MAF: now reaches M1.S9 (IN_SENS1)
- net IN_MAF: now also J1.54
- net OUT_TGV_CLOSE: now reaches M9.S2 (OUT-)
- net OUT_TGV_CLOSE: now also J1.109, J1.111
- net OUT_TGV_OPEN: now reaches M9.S3 (OUT+)
- net OUT_TGV_OPEN: now also J1.110, J1.112
- net OUT_O2_HEATER_REAR: now reaches J1.68
- net OUT_AC_RELAY: now reaches J1.99
- net OUT_MIL: now reaches J1.118
- net IN_CAM_HALL_CAM_LH: no longer names the net of M6.W2 (VR+)
- net IN_CAM_HALL_CAM_LH: no longer J1.74
Other:
- added sheet LS2 (INJ4.kicad_sch)
- added sheet LS3 (INJ4.kicad_sch)

Commit message: LSU 4.9, K-line, cruise, and option footprints for every uncertain circuit
- Front O2: Bosch LSU 4.9 on the WBO module (M3), wired as rusefi/hellen154hyundai (H- GND, H+ switched heater return to A2+A3, SEL1 to PULL_DOWN1, CAN to M1). Un/Vm/Ip reach the stock harness A33/A26/A25 through fitted 0R JP1-JP3; pads P1-P7 for a direct pigtail and external CAN. Adapter-pin table in documents/README.md.
- K-line: Hellen LIN module M10 on UART8, D20; D29 (DLC pin 6) behind open JP4.
- Cruise: main/resume/set C7/C10/C11 -> IN_D1/3/4 with 1k 1206 pull-downs; lamps A15/A16 on a 4th low-side sheet (LS4, Q17-Q20); its 2 spare channels reach EVAP A12/A13 through open JP5/JP6.
- Options (DNP, listed in bom_replace so they are not assembled): tach pull-up, FPCU command pull-up/down (series 100R fitted), FPCU status -> IN_AT2, extra cam pull-ups, neutral pull-down, fuel level pull-up; sensor ground (C31/C34/C35) selectable GND (fitted) or GNDA. Pads for spare MCU pins, rails, A22, D28, D29; prototype area G1.
- LCSC codes checked on lcsc.com (C21190, C25804, C22775, C23162, C4410, C17520, C17477).

Verified: 74 planned nets match the kicad-cli netlist exactly; whole-netlist diff shows no unplanned changes; ERC errors 235 -> 190, no new types, nothing off grid; pinout check 94 OK, 8 optional pins not wired. PCB not yet updated.

Co-Authored-By: Claude Opus 5.5 <noreply@anthropic.com>
Parts:
- removed R19, R20, R21, R22, R23: 4.7k, hellen-one-common:R0603, symbol hellen-one-common:Res
- added G1: PROTO_AREA, hellen-one-common:PROTO_AREA, symbol hellen-one-common:PROTO_AREA
- added JP1, JP2, JP3, JP8: 0R, hellen-one-common:PAD-0805-PAD, symbol hellen-one-common:Jumper-Pad-Pad
- added JP4, JP5, JP6, JP7, JP9: DNP 0R, hellen-one-common:PAD-0805-PAD, symbol hellen-one-common:Jumper-Pad-Pad
- added M10: Module-lin-0.1, hellen-one-lin-0.1:lin, symbol hellen-one-lin-0.1:Module-lin-0.1
- added P1: WBO_UN, hellen-one-common:PAD-TH, symbol hellen-one-common:Pad
- added P10: OUT_SPARE_LS2, hellen-one-common:PAD-TH, symbol hellen-one-common:Pad
- added P11: CHARGE_A22, hellen-one-common:PAD-TH, symbol hellen-one-common:Pad
- added P12: FP_STATUS, hellen-one-common:PAD-TH, symbol hellen-one-common:Pad
- added P13: DLC6_D29, hellen-one-common:PAD-TH, symbol hellen-one-common:Pad
- added P14: SPARE_INJ8, hellen-one-common:PAD-TH, symbol hellen-one-common:Pad
- added P15: SPARE_IO9, hellen-one-common:PAD-TH, symbol hellen-one-common:Pad
- added P16: SPARE_IO10, hellen-one-common:PAD-TH, symbol hellen-one-common:Pad
- added P17: SPARE_IO11, hellen-one-common:PAD-TH, symbol hellen-one-common:Pad
- added P18: SPARE_IO13, hellen-one-common:PAD-TH, symbol hellen-one-common:Pad
- added P19: +5VA, hellen-one-common:PAD-TH, symbol hellen-one-common:Pad
- added P2: WBO_VM, hellen-one-common:PAD-TH, symbol hellen-one-common:Pad
- added P20: +3.3V, hellen-one-common:PAD-TH, symbol hellen-one-common:Pad
- added P21: +12V_RAW, hellen-one-common:PAD-TH, symbol hellen-one-common:Pad
- added P22: GND, hellen-one-common:PAD-TH, symbol hellen-one-common:Pad
- added P3: WBO_IP, hellen-one-common:PAD-TH, symbol hellen-one-common:Pad
- added P4: WBO_RTRIM, hellen-one-common:PAD-TH, symbol hellen-one-common:Pad
- added P5: WBO_HEATER, hellen-one-common:PAD-TH, symbol hellen-one-common:Pad
- added P6: CAN_H, hellen-one-common:PAD-TH, symbol hellen-one-common:Pad
- added P7: CAN_L, hellen-one-common:PAD-TH, symbol hellen-one-common:Pad
- added P8: K_LINE, hellen-one-common:PAD-TH, symbol hellen-one-common:Pad
- added P9: OUT_SPARE_LS1, hellen-one-common:PAD-TH, symbol hellen-one-common:Pad
- added R30, R31, R32, R33, R34, R44: 4.7k, hellen-one-common:R0603, symbol hellen-one-common:Res
- added R35, R36, R37: 1k, hellen-one-common:R1206, symbol hellen-one-common:Res
- added R38: 2.2k, hellen-one-common:R0805, symbol hellen-one-common:Res
- added R39: 100, hellen-one-common:R0603, symbol hellen-one-common:Res
- added R40, R42, R43, R45: 1k, hellen-one-common:R0603, symbol hellen-one-common:Res
- added R41: 10k, hellen-one-common:R0603, symbol hellen-one-common:Res
Connections:
- net +12V: now also M10.N1 (12V), M10.V1 (12V)
- net +12V_RAW: now also P21.1 (Pin_1), R38.2
- net +3.3V: now also P20.1 (Pin_1)
- net +5V: now also M10.V3 (5V), R40.2
- net +5VA: now also M3.W1 (V5_IN), P19.1 (Pin_1), R42.2, R43.2, R45.2
- net FUEL_PUMP_SIGNAL1: now also R39.2, R40.1, R41.1; no longer M1.W7 (IGN5)
- net GND: now also M3.E6 (LSU_H-), M3.G (GND), JP8.2, M10.E1 (GND), M10.S1 (GND), P22.1 (Pin_1), R30.2, R31.2, R32.2, R33.2, R34.2, R35.2, R36.2, R37.2, R41.2, R44.2; no longer J1.62, J1.65, J1.66
- net GNDA: now also JP9.2
- net IN_AC_REQUEST: now also R31.1
- net IN_BRAKE_SW1: now also R34.1
- net IN_BRAKE_SW2: now also R32.1
- net IN_CAM: now also R42.1
- net IN_CAM_RH: now also R43.1
- net IN_CLUTCH: now also R33.1
- net IN_FUEL_LEVEL: now also R45.1
- net IN_NEUTRAL_SWITCH: now also R44.1
- net IN_STARTER_SWITCH: now also R30.1
- net OUT_TACH: now also R38.1
- net SPARE_IO10: now reaches M1.E10 (OUT_IO10)
- net SPARE_IO10: now also P16.1 (Pin_1)
- net SPARE_IO9: now reaches M1.E11 (OUT_IO9)
- net SPARE_IO9: now also P15.1 (Pin_1)
- net SPARE_IO13: now reaches M1.E20 (OUT_IO13)
- net SPARE_IO13: now also P18.1 (Pin_1)
- net SPARE_LS2: now reaches M1.E22 (OUT_IO8)
- net SPARE_LS1: now reaches M1.E23 (OUT_IO7)
- net SPARE_IO11: now reaches M1.E24 (OUT_IO11)
- net SPARE_IO11: now also P17.1 (Pin_1)
- net SPARE_INJ8: now reaches M1.E34 (OUT_INJ8)
- net SPARE_INJ8: now also P14.1 (Pin_1)
- net CRUISE_MAIN_LIGHT: now reaches M1.E7 (OUT_IO5)
- net CRUISE_SET_LIGHT: now reaches M1.E9 (OUT_IO6)
- net KLINE_RX: now reaches M1.N24 (UART8_RX)
- net KLINE_RX: now also M10.V2 (UART_RX)
- net KLINE_TX: now reaches M1.N25 (UART8_TX)
- net KLINE_TX: now also M10.V5 (UART_TX)
- net IN_CRUISE_SET: now reaches M1.S1 (IN_D4)
- net IN_CRUISE_SET: now also J1.42, R37.1
- net IN_CRUISE_RESUME: now reaches M1.S2 (IN_D3)
- net IN_CRUISE_RESUME: now also J1.41, R36.1
- net FP_STATUS_IN: now reaches M1.S29 (IN_AT2)
- net FP_STATUS_IN: now also JP7.2
- net IN_CRUISE_MAIN: now reaches M1.S4 (IN_D1)
- net IN_CRUISE_MAIN: now also J1.38, R35.1
- net CAN_H: now reaches M1.W12 (CANH)
- net CAN_H: now also M3.W4 (CANH), P6.1 (Pin_1)
- net CAN_L: now reaches M1.W13 (CANL)
- net CAN_L: now also M3.W3 (CANL), P7.1 (Pin_1)
- net WBO_UN: now reaches M3.E1 (LSU_Un)
- net WBO_UN: now also JP1.1, P1.1 (Pin_1)
- net WBO_VM: now reaches M3.E2 (LSU_Vm)
- net WBO_VM: now also JP2.1, P2.1 (Pin_1)
- net WBO_IP: now reaches M3.E3 (LSU_Ip)
- net WBO_IP: now also JP3.1, P3.1 (Pin_1)
- net WBO_RTRIM: now reaches M3.E4 (LSU_Rtrim)
- net WBO_RTRIM: now also P4.1 (Pin_1)
- net WBO_HEATER: now reaches M3.E5 (LSU_H+)
- net WBO_HEATER: now also J1.103, J1.104, P5.1 (Pin_1)
- net WBO_SEL1: now reaches M3.J1 (SEL1)
- net WBO_SEL1: now also M3.J_GND1 (PULL_DOWN1)
- net EVAP_A12: now reaches J1.113
- net EVAP_A12: now also JP5.2
- net EVAP_A13: now reaches J1.114
- net EVAP_A13: now also JP6.2
- net OUT_CRUISE_MAIN_LIGHT: now reaches J1.116
- net OUT_CRUISE_SET_LIGHT: now reaches J1.117
- net CHARGE_A22: now reaches J1.123
- net CHARGE_A22: now also P11.1 (Pin_1)
- net WBO_IP_J1: now reaches J1.126
- net WBO_IP_J1: now also JP3.2
- net WBO_VM_J1: now reaches J1.127
- net WBO_VM_J1: now also JP2.2
- net WBO_UN_J1: now reaches J1.134
- net WBO_UN_J1: now also JP1.2
- net K_LINE: now reaches J1.20
- net K_LINE: now also JP4.2, M10.V4 (LIN), P8.1 (Pin_1)
- net DLC6_D29: now reaches J1.29
- net DLC6_D29: now also JP4.1, P13.1 (Pin_1)
- net FUEL_PUMP_SIGNAL2 renamed FP_STATUS
- net FP_STATUS: now also JP7.1, P12.1 (Pin_1)
- new net FP_CMD: M1.W7 (IGN5), R39.1
- new net GND_SENSOR: J1.62, J1.65, J1.66, JP8.1, JP9.1
- new net OUT_SPARE_LS1: JP5.1, P9.1 (Pin_1)
- new net OUT_SPARE_LS2: JP6.1, P10.1 (Pin_1)
Other:
- added sheet LS4 (INJ4.kicad_sch)
