File: rusefiSTI2004.kicad_sch (KiCad schematic)
At the start: 68 parts, among them J1 1-1376430-0, M1 Module-mega-mcu144-0.7, M10 Module-lin-0.1, M13 Module-knock-0.2, M14 Module-power_12and5V-0.3, M2 Module-motor-driver-0.1, M3 Module-wbo-0.5, M4 Module-can-0.1, M5 Module-vr-discrete-0.5, M6 Module-vr-discrete-0.5, M7 Module-knock-0.2, M8 Module-power_12and5V-0.3, M9 Module-motor-driver-0.1, P1 WBO_UN, P10 OUT_SPARE_LS2, P11 CHARGE_A22, P12 FP_STATUS, P13 DLC6_D29, P14 SPARE_INJ8, P15 SPARE_IO9, P16 SPARE_IO10, P17 SPARE_IO11, P18 SPARE_IO13, P19 +5VA, P2 WBO_VM, P20 +3.3V, P21 +12V_RAW, P22 GND, P3 WBO_IP, P4 WBO_RTRIM, P5 WBO_HEATER, P6 CAN_H, P7 CAN_L, P8 K_LINE, P9 OUT_SPARE_LS1

Commit message: Fix board blockers; USB, boot/SWD, 8 more inputs via dinput4
Blockers found in the completeness review:
- M1 module ground GND_G was unconnected -> GND
- F5 JK-nSMD005 (50 mA PTC) in series with the throttle motor supply -> removed, D6 feeds +12V_ETB directly (car fuses the ETB relay feed)
- no USB at all -> J2 mini-B (C13453) on M1 USB D+/D-/VBUS/ID; BOOT0 pad + open JP10 to 3.3 V (DFU), SWD pads

Inputs: two Hellen dinput4 modules (M11, M12) on spare 5 V-tolerant GPIOs: defogger D11, small lights D12, blower/A-C D13, test mode D14, blow-by D24, and three aux inputs on pads (launch/2-step, map switch, spare) with pull-up/down options. I2C expander considered: rusEFI has no I2C input-expander driver and the supported MC33972 is obsolete; I2C SCL/SDA on pads for later.

Removed unused M6 (VR; cams are Hall) and M4 (CAN; M1 has a transceiver); OUT_PWM3, IN_RES2, IGN6-8 to pads.

Verified: 100 planned nets match the netlist; whole-netlist diff clean; ERC errors 190 -> 155, no new types, nothing off grid; pinout check 99 OK (only EVAP C12/C21/A24 unwired).

Co-Authored-By: Claude Opus 5.5 <noreply@anthropic.com>
Parts:
- removed F5: nSMD005, hellen-one-common:PAD-1206-PAD, symbol hellen-one-common:Fuse-Pad-Pad
- removed M4: Module-can-0.1, hellen-one-can-0.1:can, symbol hellen-one-can-0.1:Module-can-0.1
- removed M6: Module-vr-discrete-0.5, hellen-one-vr-discrete-0.5:vr-discrete, symbol hellen-one-vr-discrete-0.5:Module-vr-discrete-0.5
- added J2: USB_B_Mini, hellen-one-common:USB-MINI-B-VERTICAL, symbol hellen-one-common:USB_B_Mini
- added JP10: DNP 0R, hellen-one-common:PAD-0805-PAD, symbol hellen-one-common:Jumper-Pad-Pad
- added M11, M12: Module-dinput4-0.1, hellen-one-dinput4-0.1:dinput4, symbol hellen-one-dinput4-0.1:Module-dinput4-0.1
- added P23: BOOT0, hellen-one-common:PAD-TH, symbol hellen-one-common:Pad
- added P24: SWDIO, hellen-one-common:PAD-TH, symbol hellen-one-common:Pad
- added P25: SWCLK, hellen-one-common:PAD-TH, symbol hellen-one-common:Pad
- added P26: NRST, hellen-one-common:PAD-TH, symbol hellen-one-common:Pad
- added P27: SPARE_PWM3, hellen-one-common:PAD-TH, symbol hellen-one-common:Pad
- added P28: SPARE_RES2, hellen-one-common:PAD-TH, symbol hellen-one-common:Pad
- added P29: AUX_IN1, hellen-one-common:PAD-TH, symbol hellen-one-common:Pad
- added P30: AUX_IN2, hellen-one-common:PAD-TH, symbol hellen-one-common:Pad
- added P31: AUX_IN3, hellen-one-common:PAD-TH, symbol hellen-one-common:Pad
- added R46, R47, R48: 4.7k, hellen-one-common:R0603, symbol hellen-one-common:Res
- added R49, R50, R51: 10k, hellen-one-common:R0603, symbol hellen-one-common:Res
- P14: value SPARE_INJ8 -> SPARE_IGN6
- P15: value SPARE_IO9 -> SPARE_IGN7
- P16: value SPARE_IO10 -> SPARE_IGN8
- P17: value SPARE_IO11 -> I2C_SCL
- P18: value SPARE_IO13 -> I2C_SDA
Connections:
- net +12V_ETB: now also J1.6
- net +3.3V: now also JP10.2
- net +5V: now also M11.J1 (PULL_D1), M11.J2 (PULL_D2), M11.J3 (PULL_D3), M11.J4 (PULL_D4), M11.V1 (V5), M12.J4 (PULL_D4), M12.V1 (V5), R49.2, R50.2, R51.2
- net GND: now also M1.G (GND), J2.5 (GND), J2.6 (Shield), M11.G (GND), M12.G (GND), M12.J1 (PULL_D1), M12.J2 (PULL_D2), M12.J3 (PULL_D3), R46.2, R47.2, R48.2
- net DIN_SMALL_LIGHT: now reaches M1.E35 (IO6)
- net DIN_SMALL_LIGHT: now also M11.W3 (OUT_D2)
- net DIN_BLOWER: now reaches M1.E36 (IO7)
- net DIN_BLOWER: now also M11.W2 (OUT_D3)
- net USB_ID: now reaches M1.N1 (USBID)
- net USB_ID: now also J2.4 (ID)
- net I2C_SCL: now reaches M1.N14 (I2C_SCL)
- net I2C_SCL: now also P17.1 (Pin_1)
- net I2C_SDA: now reaches M1.N15 (I2C_SDA)
- net I2C_SDA: now also P18.1 (Pin_1)
- net USB_DM: now reaches M1.N2 (USBM)
- net USB_DM: now also J2.2 (D-)
- net DIN_DEFOG: now reaches M1.N23 (IO5)
- net DIN_DEFOG: now also M11.W4 (OUT_D1)
- net USB_DP: now reaches M1.N3 (USBP)
- net USB_DP: now also J2.3 (D+)
- net USB_VBUS: now reaches M1.N4 (VBUS)
- net USB_VBUS: now also J2.1 (VBUS)
- net BOOT0: now reaches M1.N5 (BOOT0)
- net BOOT0: now also JP10.1, P23.1 (Pin_1)
- net SWDIO: now reaches M1.N7 (SWDIO)
- net SWDIO: now also P24.1 (Pin_1)
- net SWCLK: now reaches M1.N8 (SWCLK)
- net SWCLK: now also P25.1 (Pin_1)
- net NRST: now reaches M1.N9 (nReset)
- net NRST: now also P26.1 (Pin_1)
- net SPARE_IGN8: now reaches M1.W4 (IGN8)
- net SPARE_IGN8: now also P16.1 (Pin_1)
- net SPARE_IGN7: now reaches M1.W5 (IGN7)
- net SPARE_IGN7: now also P15.1 (Pin_1)
- net SPARE_IGN6: now reaches M1.W6 (IGN6)
- net SPARE_IGN6: now also P14.1 (Pin_1)
- net IN_DEFOG: now reaches J1.11
- net IN_DEFOG: now also M11.V2 (IN_D1), R49.1
- net IN_SMALL_LIGHT: now reaches J1.12
- net IN_SMALL_LIGHT: now also M11.V3 (IN_D2), R50.1
- net IN_BLOWER: now reaches J1.13
- net IN_BLOWER: now also M11.V4 (IN_D3), R51.1
- net IN_TEST_MODE: now reaches J1.14
- net IN_TEST_MODE: now also M11.V5 (IN_D4)
- net IN_BLOWBY: now reaches J1.24
- net IN_BLOWBY: now also M12.V5 (IN_D4)
- net SPARE_INJ8 renamed DIN_BLOWBY
- net DIN_BLOWBY: now also M12.W1 (OUT_D4); no longer P14.1 (Pin_1)
- net SPARE_IO10 renamed DIN_AUX2
- net DIN_AUX2: now also M12.W3 (OUT_D2); no longer P16.1 (Pin_1)
- net SPARE_IO11 renamed DIN_AUX3
- net DIN_AUX3: now also M12.W2 (OUT_D3); no longer P17.1 (Pin_1)
- net SPARE_IO13 renamed DIN_TEST_MODE
- net DIN_TEST_MODE: now also M11.W1 (OUT_D4); no longer P18.1 (Pin_1)
- net SPARE_IO9 renamed DIN_AUX1
- net DIN_AUX1: now also M12.W4 (OUT_D1); no longer P15.1 (Pin_1)
- net THRESHOLD_VR_CAM renamed SPARE_PWM3
- net SPARE_PWM3: now also P27.1 (Pin_1)
- net VR_ANALOG_CAM renamed SPARE_RES2
- net SPARE_RES2: now also P28.1 (Pin_1)
- new net AUX_IN1: M12.V2 (IN_D1), P29.1 (Pin_1), R46.1
- new net AUX_IN2: M12.V3 (IN_D2), P30.1 (Pin_1), R47.1
- new net AUX_IN3: M12.V4 (IN_D3), P31.1 (Pin_1), R48.1

Commit message: Own 5 V for the pedal, CAN terminator option, Mini-Fit Jr aux connector
- Pedal supply C15 (APS_PS_5V) now from the second power module M8's protected 5 V; C16 sensor 5 V stays on M14. M8 fed like M14 (+12V_RAW, +12V_IGN, +12V_BACK_UP, PWR_EN). Open JP11 falls back to +5VAS; M8 power-good on pad P32.
- CAN: M1 terminates internally (R100 120R); WBO has none. R52 120R (DNP) at the aux connector for an external bus end.
- J3 aux connector, Molex Mini-Fit Jr 5566-14A 2x7 vertical (39281143): +12 V via F6 0.5 A PTC, +5 V sensor via F7 50 mA PTC, sensor ground, AUX_IN1-3 (launch/2-step, map switch, spare), AUX_AN1 (IN_RES2), AUX_AN2 (IN_AT2, shared with the FPCU status option), two low-side outputs, CAN H/L, 2x GND. Symbol and footprint from KiCad 8.0.7 libs; footprint copied into STI.pretty.

Verified: 104 planned nets match the netlist; whole-netlist diff clean; ERC errors 155 -> 148, no new types; pinout check 99 OK.

Co-Authored-By: Claude Opus 5.5 <noreply@anthropic.com>
Parts:
- added F6: nSMD050-24V, hellen-one-common:PAD-1206-PAD, symbol hellen-one-common:Fuse-Pad-Pad
- added F7: nSMD005, hellen-one-common:PAD-1206-PAD, symbol hellen-one-common:Fuse-Pad-Pad
- added J3: MiniFitJr_2x07_AUX, STI:Molex_Mini-Fit_Jr_5566-14A_2x07_P4.20mm_Vertical, symbol Connector_Generic:Conn_02x07_Odd_Even
- added JP11: DNP 0R, hellen-one-common:PAD-0805-PAD, symbol hellen-one-common:Jumper-Pad-Pad
- added P32: PG_5VP_APS, hellen-one-common:PAD-TH, symbol hellen-one-common:Pad
- added R52: 120, hellen-one-common:R0603, symbol hellen-one-common:Res
Connections:
- net +12V_BACK_UP: now also M8.V1 (V12_PERM)
- net +12V_IGN: now also M8.V2 (IN_VIGN)
- net +12V_RAW: now also M8.V3 (V12_RAW), F6.1
- net +5VAS: now also F7.1, JP11.2; no longer J1.46
- net AUX_IN1: now also J3.5 (Pin_5)
- net AUX_IN2: now also J3.6 (Pin_6)
- net AUX_IN3: now also J3.7 (Pin_7)
- net CAN_H: now also J3.12 (Pin_12), R52.1
- net CAN_L: now also J3.13 (Pin_13), R52.2
- net GND: now also M8.S1 (GND), J3.14 (Pin_14), J3.2 (Pin_2)
- net GND_SENSOR: now also J3.4 (Pin_4)
- net OUT_SPARE_LS1: now also J3.10 (Pin_10)
- net OUT_SPARE_LS2: now also J3.11 (Pin_11)
- net PWR_EN: now also M8.E5 (EN_5VP)
- net SPARE_RES2: now also J3.8 (Pin_8)
- net PG_5VP_APS: now reaches M8.E6 (PG_5VP)
- net PG_5VP_APS: now also P32.1 (Pin_1)
- net APS_PS_5V: now reaches M8.V4 (5VP)
- net APS_PS_5V: now also J1.46, JP11.1
- net FP_STATUS_IN renamed AUX_AN2
- net AUX_AN2: now also J3.9 (Pin_9)
- new net AUX_12V: F6.2, J3.1 (Pin_1)
- new net AUX_5V: F7.2, J3.3 (Pin_3)

Commit message: No overlapping text; USB-C; KiCad 8 compatibility checked
- tools/sch_overlap_check.py: fails on any label/field/sheet text overlapping other text or a symbol body (KiCad stroke-font estimate, field angles relative to the symbol).
- Layout rules in the generator: power symbols point along their wire with horizontal names; adjacent same-rail pins share one symbol; labels follow pin direction; module names above the body; small parts placed by a collision-checked search; a final pass moves any touching field; the build fails unless overlaps = 0. Original-sheet overlaps fixed too.
- USB: J2 is now the EmbeddedEra library USB-C (HRO TYPE-C-31-M-12, C165948) with 5.1k CC pull-downs, USBLC6-2SC6 ESD (C7519), shield via fitted 0R. Footprints copied into STI.pretty and converted to KiCad 8 syntax.
- Imported symbols converted from KiCad 10 to KiCad 8 syntax (hide flags, dropped 9/10-only tokens).

Verified: netlist connectivity identical to the previous commit apart from the USB change; KiCad 8.0.7 (Hellen CI) and KiCad 10 give the same connectivity; ERC no new error types; 0 overlaps.

Co-Authored-By: Claude Opus 5.5 <noreply@anthropic.com>
Parts:
- removed J2: USB_B_Mini, hellen-one-common:USB-MINI-B-VERTICAL, symbol hellen-one-common:USB_B_Mini
- added J2: USB C 2.0 16P, STI:USB_C_Receptacle_HRO_TYPE-C-31-M-12, symbol EmbeddedEra_Neoden_YY1_PNP:USB_C_Receptacle_USB2.0_16P
- added JP12: DNP 0R, hellen-one-common:PAD-0805-PAD, symbol hellen-one-common:Jumper-Pad-Pad
- added R53: 10k, hellen-one-common:R0603, symbol hellen-one-common:Res
- added R54: 120, hellen-one-common:R0603, symbol hellen-one-common:Res
- added U1: USBLC6-2SC6, STI:SOT-23-6, symbol EmbeddedEra:USBLC6-2P6
- JP10: value DNP 0R -> 0R; now fitted
- R46, R47: value 4.7k -> 5.1k; LCSC C23162 -> C23186; now fitted
- R49, R50: value 10k -> 4.7k; LCSC C25804 -> C23162
- R52: value 120 -> 10k; LCSC C22787 -> C25804
Connections:
- net +3.3V: now also JP11.2; no longer JP10.2
- net +5V: now also R52.2, R53.2; no longer R49.2, R50.2
- net +5VAS: now also JP12.2; no longer JP11.2
- net APS_PS_5V: now also JP12.1; no longer JP11.1
- net AUX_IN1: now also R48.1; no longer R46.1
- net AUX_IN2: now also R49.1; no longer R47.1
- net AUX_IN3: now also R50.1; no longer R48.1
- net BOOT0: now also JP11.1; no longer JP10.1
- net CAN_H: now also R54.1; no longer R52.1
- net CAN_L: now also R54.2; no longer R52.2
- net GND: now also JP10.2, R49.2, R50.2, J2.A1 (GND), J2.A12 (GND), J2.B1 (GND), J2.B12 (GND), U1.2 (GND)
- net IN_BLOWER: now also R53.1; no longer R51.1
- net IN_DEFOG: now also R51.1; no longer R49.1
- net IN_SMALL_LIGHT: now also R52.1; no longer R50.1
- net USB_DM: now also J2.A7 (D-), J2.B7 (D-), U1.3 (I/O2), U1.4 (I/O2)
- net USB_DP: now also J2.A6 (D+), J2.B6 (D+), U1.1 (I/O1), U1.6 (I/O1)
- net USB_VBUS: now also J2.A4 (VBUS), J2.A9 (VBUS), J2.B4 (VBUS), J2.B9 (VBUS), U1.5 (VBUS)
- net USB_ID: no longer names the net of M1.N1 (USBID)
- new net USB_CC1: J2.A5 (CC1), R46.1
- new net USB_CC2: J2.B5 (CC2), R47.1
- new net USB_SHIELD: J2.S1 (SHIELD), JP10.1

Commit message: Split the schematic into functional sheets with notes
Root page is now an overview (block per sheet, how to read it). Sheets: Vehicle connector (J1, all four plugs), Power (M14, M8 pedal 5 V), MCU and USB, Sensors, Switch inputs, Outputs (low-side sheets INJ/LS1-LS4 nested here, throttle, TGV, fuel pump), Comms (LSU 4.9 WBO, K-line, CAN), Aux and expansion (J3, spares, proto area). Each sheet opens with a note on what it holds and why.

Labels that name a net are global labels (pointing away from their wire); descriptive labels on power nets stay local so GND keeps its name. tools/options_table.py generates the option-parts table in documents/README.md from the schematic.

Verified: connectivity and every net name identical to the flat schematic (167 nets), in KiCad 10 and KiCad 8.0.7; 0 text overlaps on all 10 sheet files; ERC unchanged (no-connects added on unused USB-C SBU and MCU USBID); pinout check 99 OK.

Co-Authored-By: Claude Opus 5.5 <noreply@anthropic.com>
Parts:
- removed F1, F2, F3, F4, F7: nSMD005, hellen-one-common:PAD-1206-PAD, symbol hellen-one-common:Fuse-Pad-Pad
- removed F6: nSMD050-24V, hellen-one-common:PAD-1206-PAD, symbol hellen-one-common:Fuse-Pad-Pad
- removed G1: PROTO_AREA, hellen-one-common:PROTO_AREA, symbol hellen-one-common:PROTO_AREA
- removed J1: 1-1376430-0, STI:1-1376430-0, symbol rusefi_1-1376430-0_135pin:1-1376430-0
- removed J2: USB C 2.0 16P, STI:USB_C_Receptacle_HRO_TYPE-C-31-M-12, symbol EmbeddedEra_Neoden_YY1_PNP:USB_C_Receptacle_USB2.0_16P
- removed J3: MiniFitJr_2x07_AUX, STI:Molex_Mini-Fit_Jr_5566-14A_2x07_P4.20mm_Vertical, symbol Connector_Generic:Conn_02x07_Odd_Even
- removed JP1, JP10, JP2, JP3, JP8: 0R, hellen-one-common:PAD-0805-PAD, symbol hellen-one-common:Jumper-Pad-Pad
- removed JP11, JP12, JP4, JP5, JP6, JP7, JP9: DNP 0R, hellen-one-common:PAD-0805-PAD, symbol hellen-one-common:Jumper-Pad-Pad
- removed M1: Module-mega-mcu144-0.7, hellen-one-mega-mcu144-0.7:mega-mcu144, symbol hellen-one-mega-mcu144-0.7:Module-mega-mcu144-0.7
- removed M10: Module-lin-0.1, hellen-one-lin-0.1:lin, symbol hellen-one-lin-0.1:Module-lin-0.1
- removed M11, M12: Module-dinput4-0.1, hellen-one-dinput4-0.1:dinput4, symbol hellen-one-dinput4-0.1:Module-dinput4-0.1
- removed M13, M7: Module-knock-0.2, hellen-one-knock-0.2:knock, symbol hellen-one-knock-0.2:Module-knock-0.2
- removed M14, M8: Module-power_12and5V-0.3, hellen-one-power_12and5V-0.3:power_12and5V, symbol hellen-one-power_12and5V-0.3:Module-power_12and5V-0.3
- removed M2, M9: Module-motor-driver-0.1, hellen-one-motor-driver-0.1:motor-driver, symbol hellen-one-motor-driver-0.1:Module-motor-driver-0.1
- removed M3: Module-wbo-0.5, hellen-one-wbo-0.5:wbo, symbol hellen-one-wbo-0.5:Module-wbo-0.5
- removed M5: Module-vr-discrete-0.5, hellen-one-vr-discrete-0.5:vr-discrete, symbol hellen-one-vr-discrete-0.5:Module-vr-discrete-0.5
- removed P1: WBO_UN, hellen-one-common:PAD-TH, symbol hellen-one-common:Pad
- removed P10: OUT_SPARE_LS2, hellen-one-common:PAD-TH, symbol hellen-one-common:Pad
- removed P11: CHARGE_A22, hellen-one-common:PAD-TH, symbol hellen-one-common:Pad
- removed P12: FP_STATUS, hellen-one-common:PAD-TH, symbol hellen-one-common:Pad
- removed P13: DLC6_D29, hellen-one-common:PAD-TH, symbol hellen-one-common:Pad
- removed P14: SPARE_IGN6, hellen-one-common:PAD-TH, symbol hellen-one-common:Pad
- removed P15: SPARE_IGN7, hellen-one-common:PAD-TH, symbol hellen-one-common:Pad
- removed P16: SPARE_IGN8, hellen-one-common:PAD-TH, symbol hellen-one-common:Pad
- removed P17: I2C_SCL, hellen-one-common:PAD-TH, symbol hellen-one-common:Pad
- removed P18: I2C_SDA, hellen-one-common:PAD-TH, symbol hellen-one-common:Pad
- removed P19: +5VA, hellen-one-common:PAD-TH, symbol hellen-one-common:Pad
- removed P2: WBO_VM, hellen-one-common:PAD-TH, symbol hellen-one-common:Pad
- removed P20: +3.3V, hellen-one-common:PAD-TH, symbol hellen-one-common:Pad
- removed P21: +12V_RAW, hellen-one-common:PAD-TH, symbol hellen-one-common:Pad
- removed P22: GND, hellen-one-common:PAD-TH, symbol hellen-one-common:Pad
- removed P23: BOOT0, hellen-one-common:PAD-TH, symbol hellen-one-common:Pad
- removed P24: SWDIO, hellen-one-common:PAD-TH, symbol hellen-one-common:Pad
- removed P25: SWCLK, hellen-one-common:PAD-TH, symbol hellen-one-common:Pad
- removed P26: NRST, hellen-one-common:PAD-TH, symbol hellen-one-common:Pad
- removed P27: SPARE_PWM3, hellen-one-common:PAD-TH, symbol hellen-one-common:Pad
- removed P28: SPARE_RES2, hellen-one-common:PAD-TH, symbol hellen-one-common:Pad
- removed P29: AUX_IN1, hellen-one-common:PAD-TH, symbol hellen-one-common:Pad
- removed P3: WBO_IP, hellen-one-common:PAD-TH, symbol hellen-one-common:Pad
- removed P30: AUX_IN2, hellen-one-common:PAD-TH, symbol hellen-one-common:Pad
- removed P31: AUX_IN3, hellen-one-common:PAD-TH, symbol hellen-one-common:Pad
- removed P32: PG_5VP_APS, hellen-one-common:PAD-TH, symbol hellen-one-common:Pad
- removed P4: WBO_RTRIM, hellen-one-common:PAD-TH, symbol hellen-one-common:Pad
- removed P5: WBO_HEATER, hellen-one-common:PAD-TH, symbol hellen-one-common:Pad
- removed P6: CAN_H, hellen-one-common:PAD-TH, symbol hellen-one-common:Pad
- removed P7: CAN_L, hellen-one-common:PAD-TH, symbol hellen-one-common:Pad
- removed P8: K_LINE, hellen-one-common:PAD-TH, symbol hellen-one-common:Pad
- removed P9: OUT_SPARE_LS1, hellen-one-common:PAD-TH, symbol hellen-one-common:Pad
- removed R1: 33k, hellen-one-common:R0603, symbol hellen-one-common:Res
- removed R2: 6.8k, hellen-one-common:R0603, symbol hellen-one-common:Res
- removed R30, R31, R32, R33, R34, R44, R48, R49, R50: 4.7k, hellen-one-common:R0603, symbol hellen-one-common:Res
- removed R35, R36, R37: 1k, hellen-one-common:R1206, symbol hellen-one-common:Res
- removed R38: 2.2k, hellen-one-common:R0805, symbol hellen-one-common:Res
- removed R39: 100, hellen-one-common:R0603, symbol hellen-one-common:Res
- removed R40, R42, R43, R45: 1k, hellen-one-common:R0603, symbol hellen-one-common:Res
- removed R41, R51, R52, R53: 10k, hellen-one-common:R0603, symbol hellen-one-common:Res
- removed R46, R47: 5.1k, hellen-one-common:R0603, symbol hellen-one-common:Res
- removed R54: 120, hellen-one-common:R0603, symbol hellen-one-common:Res
- removed U1: USBLC6-2SC6, STI:SOT-23-6, symbol EmbeddedEra:USBLC6-2P6
Other:
- removed sheet INJ
- removed sheet LS1
- removed sheet LS2
- removed sheet LS3
- removed sheet LS4
- added sheet Aux and expansion (Aux.kicad_sch)
- added sheet Comms (Comms.kicad_sch)
- added sheet MCU and USB (Mcu.kicad_sch)
- added sheet Outputs (Outputs.kicad_sch)
- added sheet Power (Power.kicad_sch)
- added sheet Sensors (Sensors.kicad_sch)
- added sheet Switch inputs (Inputs.kicad_sch)
- added sheet Vehicle connector (Connector.kicad_sch)
- note added: "Built from Hellen-One modules. Signals between sheets are global net labels; power symbols are global. Crossed-out (DNP) parts are optional footprints, not assembled: what each one is for is in documents/README.md. Car pinout and cross-check: documents/STI2004-pinout-check.xlsx (tools/pinout_check.py). Sheet order follows the signal: car connector -> power -> MCU -> inputs -> outputs -> comms -> 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"
- note added: "Crank: 2-wire VR sensor (B10 +, B22 -) into M5. Knock (C25) into M13. M7 is a spare knock channel (not used)."
- note added: "J3: Molex Mini-Fit Jr 2x7 (pinout in documents/README.md): fused 12 V and 5 V, sensor ground, three digital"
- note added: "Low-side drivers (VND14NV04) in sub-sheets: INJ injectors 1-4; LS1 main relay, fans, ETB relay;"
- note added: "M11/M12 (dinput4): car lines that close to ground (defogger D11, lights D12, blower D13, test mode D14,"
- note added: "M14 (main power module): +12V_RAW from the main relay (B5/B6), +12V_IGN (D15), back-up +12V (B19)."
- note added: "M1: Hellen mega-mcu144 (STM32F7), with a 120R CAN terminator built in."
- note added: "M3: rusEFI wideband (WBO) for a Bosch LSU 4.9 front O2, on CAN to M1. It reaches the sensor through the stock"
- note added: "Units: D = B137, C = B136, B = B135, A = B134. Every pin carries a global net label used on the other sheets."
- note added: "rusEFI STI 2004: plug-and-play ECU for the 2004 USDM Subaru Impreza WRX STI (EJ257, drive-by-wire)."
- note removed: "A: B134"
- note removed: "B: B135"
- note removed: "C: B136"
- note removed: "D: B137"
