File: Comms.kicad_sch (KiCad schematic)
At the start: 16 parts, among them M10 Module-lin-0.1, M3 Module-wbo-0.5, P1 WBO_UN, P13 DLC6_D29, P2 WBO_VM, P3 WBO_IP, P4 WBO_RTRIM, P5 WBO_HEATER, P6 CAN_H, P7 CAN_L, P8 K_LINE

Commit message: EmbeddedEra libraries and template, KiCad 10
- Every symbol except the nine Hellen-One modules now comes from the EmbeddedEra library (resistors and 0R links from the generic libraries, PTC fuses, VND14NV04-E, TE 1-1376430-0, Molex 39281143, test pads, proto area, power symbols). Same-pin parts swapped in place; resistors re-placed between their old pin points with short wires. New parts live on library branch sti2004-parts.
- EmbeddedEra project template: worksheet, text variables, net classes with explicit power classes, JLCPCB design rules; template net names for USB, I2C and the K-line UART.
- Migrated all sheets and the board to KiCad 10 (10.0.7).
- tools/sch_overlap_check.py also fails on overlapping symbol bodies and on fields printed across a wire (found the stacked PTC fuses); KiCad 10 hide flags understood.

Verified: connectivity identical to the previous commit (167 nets), only the planned net renames; 0 overlaps on all 10 sheet files; ERC errors unchanged (148); pinout check 99 OK.

Co-Authored-By: Claude Opus 5.5 <noreply@anthropic.com>
Parts:
- removed JP1, JP2, JP3: 0R, hellen-one-common:PAD-0805-PAD, symbol hellen-one-common:Jumper-Pad-Pad
- removed JP4: DNP 0R, hellen-one-common:PAD-0805-PAD, symbol hellen-one-common:Jumper-Pad-Pad
- removed P1: WBO_UN, hellen-one-common:PAD-TH, symbol hellen-one-common:Pad
- removed P13: DLC6_D29, hellen-one-common:PAD-TH, symbol hellen-one-common:Pad
- removed P2: WBO_VM, hellen-one-common:PAD-TH, symbol hellen-one-common:Pad
- removed P3: WBO_IP, hellen-one-common:PAD-TH, symbol hellen-one-common:Pad
- removed P4: WBO_RTRIM, hellen-one-common:PAD-TH, symbol hellen-one-common:Pad
- removed P5: WBO_HEATER, hellen-one-common:PAD-TH, symbol hellen-one-common:Pad
- removed P6: CAN_H, hellen-one-common:PAD-TH, symbol hellen-one-common:Pad
- removed P7: CAN_L, hellen-one-common:PAD-TH, symbol hellen-one-common:Pad
- removed P8: K_LINE, hellen-one-common:PAD-TH, symbol hellen-one-common:Pad
- removed R54: 120, hellen-one-common:R0603, symbol hellen-one-common:Res
- added JP1, JP2, JP3, JP4: 0, EmbeddedEra_Library:R_0805_2012Metric, symbol EmbeddedEra_Resistors_0805_5pct:EE_R_0805_0_5%
- added P1: WBO_UN, EmbeddedEra_Library:TestPoint_THTPad_D2.0mm_Drill1.0mm, symbol EmbeddedEra:TestPoint_THT
- added P13: DLC6_D29, EmbeddedEra_Library:TestPoint_THTPad_D2.0mm_Drill1.0mm, symbol EmbeddedEra:TestPoint_THT
- added P2: WBO_VM, EmbeddedEra_Library:TestPoint_THTPad_D2.0mm_Drill1.0mm, symbol EmbeddedEra:TestPoint_THT
- added P3: WBO_IP, EmbeddedEra_Library:TestPoint_THTPad_D2.0mm_Drill1.0mm, symbol EmbeddedEra:TestPoint_THT
- added P4: WBO_RTRIM, EmbeddedEra_Library:TestPoint_THTPad_D2.0mm_Drill1.0mm, symbol EmbeddedEra:TestPoint_THT
- added P5: WBO_HEATER, EmbeddedEra_Library:TestPoint_THTPad_D2.0mm_Drill1.0mm, symbol EmbeddedEra:TestPoint_THT
- added P6: CAN_H, EmbeddedEra_Library:TestPoint_THTPad_D2.0mm_Drill1.0mm, symbol EmbeddedEra:TestPoint_THT
- added P7: CAN_L, EmbeddedEra_Library:TestPoint_THTPad_D2.0mm_Drill1.0mm, symbol EmbeddedEra:TestPoint_THT
- added P8: K_LINE, EmbeddedEra_Library:TestPoint_THTPad_D2.0mm_Drill1.0mm, symbol EmbeddedEra:TestPoint_THT
- added R54: 120, EmbeddedEra_Library:R_0603_1608Metric, symbol EmbeddedEra_Resistors_0603:EE_R_0603_120_1%
Connections:
- net CAN_H: now also P6.1, R54.1
- net CAN_L: now also P7.1, R54.2
- net DLC6_D29: now also JP4.1, P13.1
- net K_LINE: now also JP4.2, P8.1
- net WBO_HEATER: now also P5.1
- net WBO_IP: now also JP3.1, P3.1
- net WBO_IP_J1: now also JP3.2
- net WBO_RTRIM: now also P4.1
- net WBO_UN: now also JP1.1, P1.1
- net WBO_UN_J1: now also JP1.2
- net WBO_VM: now also JP2.1, P2.1
- net WBO_VM_J1: now also JP2.2
- net KLINE_RX renamed UART_8_RX
- net KLINE_TX renamed UART_8_TX
