File: Comms.kicad_sch (KiCad schematic)
At the start: 16 parts, among them M10 Module-lin-0.1, M3 Module-wbo-0.5, P1 WBO_UN, P13 DLC6_D29, P2 WBO_VM, P3 WBO_IP, P4 WBO_RTRIM, P5 WBO_HEATER, P6 CAN_H, P7 CAN_L, P8 K_LINE

Commit message: U1 is the library USBLC6-2SC6 (EE-C-0146); J2 part numbers; test pads and proto area out of the BOM
- U1 used the USBLC6-2P6 (SOT-666) symbol with a hand-changed footprint; now EmbeddedEra:USBLC6-2SC6.
- J2 instance had no Manufacturer/MPN although the library has them.
- P1-P32 and G1 are pads, nothing is bought (SOP-008 step 18): in_bom no, as in the library.

Co-Authored-By: Claude Opus 5.5 <noreply@anthropic.com>
Parts:
- P1, P13, P2, P3, P4, P5, P6, P7, P8: now left out of the parts list
Changed lines of the file:
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@@
 		(body_style 1)
 		(exclude_from_sim no)
-		(in_bom yes)
+		(in_bom no)
 		(on_board yes)
 		(in_pos_files yes)
@@
 		(body_style 1)
 		(exclude_from_sim no)
-		(in_bom yes)
+		(in_bom no)
 		(on_board yes)
 		(in_pos_files yes)
@@
 		(body_style 1)
 		(exclude_from_sim no)
-		(in_bom yes)
+		(in_bom no)
 		(on_board yes)
 		(in_pos_files yes)
@@
 		(body_style 1)
 		(exclude_from_sim no)
-		(in_bom yes)
+		(in_bom no)
 		(on_board yes)
 		(in_pos_files yes)
@@
 		(body_style 1)
 		(exclude_from_sim no)
-		(in_bom yes)
+		(in_bom no)
 		(on_board yes)
 		(in_pos_files yes)
@@
 		(body_style 1)
 		(exclude_from_sim no)
-		(in_bom yes)
+		(in_bom no)
 		(on_board yes)
 		(in_pos_files yes)
@@
 		(body_style 1)
 		(exclude_from_sim no)
-		(in_bom yes)
+		(in_bom no)
 		(on_board yes)
 		(in_pos_files yes)
@@
 		(body_style 1)
 		(exclude_from_sim no)
-		(in_bom yes)
+		(in_bom no)
 		(on_board yes)
 		(in_pos_files yes)
@@
 		(body_style 1)
 		(exclude_from_sim no)
-		(in_bom yes)
+		(in_bom no)
 		(on_board yes)
 		(in_pos_files yes)

Commit message: Title block: TITLE is the project name (${Project_Name}) on every sheet, DESCRIPTION the sheet name
The LS/INJ sub-sheet and the root had no title at all.

Co-Authored-By: Claude Opus 5.5 <noreply@anthropic.com>
Other:
- title: Comms -> ${Project_Name}
Changed lines of the file:
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@@
 	(paper "A3")
 	(title_block
-		(title "Comms")
+		(title "${Project_Name}")
 		(date "2026-10-13")
 	)

Commit message: WBO module M3 0.5 -> 0.6: one heater pin LSU_Htr (E5, WBO_HEATER), E6/GND removed
Evidence: hellen-one wbo/0.6 schematic (Q600 drain -> E5, source -> GND on module); rusefi/uaefi wires only E5 to the heater net (no GND on a second pin).
Netlist diff: only GND loses M3 E6; WBO_HEATER unchanged (J1 103/104, M3 E5, P5).
ERC 371 -> 370 (the removed GND symbol), nothing new; overlaps 0 on all 12 sheets; kicad-tidy-check netlist 294 nets 0 changed.
sym-lib-table: wbo 0.6; fp-lib-table: 0.6 added, 0.5 kept (PCB still uses it until the floorplan rebuild).

Co-Authored-By: Claude Sonnet 5.5 <noreply@anthropic.com>
Parts:
- M3: value Module-wbo-0.5 -> Module-wbo-0.6; footprint hellen-one-wbo-0.5:wbo -> hellen-one-wbo-0.6:wbo; symbol hellen-one-wbo-0.5:Module-wbo-0.5 -> hellen-one-wbo-0.6:Module-wbo-0.6
Connections:
- net GND: no longer M3.E6 (LSU_H-)
Changed lines of the file:
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@@
-	(wire
-		(pts
-			(xy 80.01 55.88) (xy 85.09 55.88)
-		)
-		(stroke
-			(width 0)
-			(type default)
-		)
-	)
 	(wire
 		(pts
@@
 		)
 	)
-	(symbol
-		(lib_id "EmbeddedEra_Generic:GND")
-		(at 85.09 55.88 90)
-		(unit 1)
-		(body_style 1)
-		(exclude_from_sim no)
-		(in_bom yes)
-		(on_board yes)
-		(in_pos_files yes)
-		(dnp no)
-		(property "Reference" "#PWR070"
-			(at 85.09 55.88 270)
-			(hide yes)
-			(show_name no)
-			(do_not_autoplace no)
-			(effects
-				(font
-					(size 1.27 1.27)
-				)
-			)
-		)
-		(property "Value" "GND"
-			(at 88.9 55.88 270)
-			(show_name no)
-			(do_not_autoplace no)
-			(effects
-				(font
-					(size 1.27 1.27)
-				)
-				(justify left)
-			)
-		)
-		(property "Footprint" ""
-			(at 85.09 55.88 270)
-			(hide yes)
-			(show_name no)
-			(do_not_autoplace no)
-			(effects
-				(font
-					(size 1.27 1.27)
-				)
-			)
-		)
-		(property "Datasheet" ""
-			(at 85.09 55.88 270)
-			(hide yes)
-			(show_name no)
-			(do_not_autoplace no)
-			(effects
-				(font
-					(size 1.27 1.27)
-				)
-			)
-		)
-		(property "Description" "Power symbol creates a global label with name \"GND\" , ground. Copied from KiCad library power:GND (KiCad 10.0), CC-BY-SA 4.0 with the KiCad library exception."
-			(at 85.09 55.88 270)
-			(hide yes)
-			(show_name no)
-			(do_not_autoplace no)
-			(effects
-				(font
-					(size 1.27 1.27)
-				)
-			)
-		)
-		(pin "1"
-		)
-		(instances
-			(project "rusefiSTI2004"
-				(path "/00d4d98c-a749-4bd2-a087-ea484becbbe4/b698161d-5eaf-5046-aa12-9fab6361af26"
-					(reference "#PWR070")
-					(unit 1)
-				)
-			)
-		)
-	)
-	(symbol
+(symbol
 		(lib_id "EmbeddedEra:TestPoint_THT")
 		(at 30.48 104.14 270)
@@
 	)
 	(symbol
-		(lib_id "hellen-one-wbo-0.5:Module-wbo-0.5")
+		(lib_id "hellen-one-wbo-0.6:Module-wbo-0.6")
 		(at 39.37 50.8 0)
 		(unit 1)
@@
 			)
 		)
-		(property "Value" "Module-wbo-0.5"
+		(property "Value" "Module-wbo-0.6"
 			(at 55.88 48.26 0)
 			(show_name no)
@@
 			)
 		)
-		(property "Footprint" "hellen-one-wbo-0.5:wbo"
+		(property "Footprint" "hellen-one-wbo-0.6:wbo"
 			(at 64.77 49.53 0)
 			(hide yes)
@@
 		(pin "W1"
 		)
-		(pin "E6"
-		)
-		(pin "W2"
+	(pin "W2"
 		)
 		(pin "J_VCC2"
