File: Inputs.kicad_sch (KiCad schematic)
At the start: 15 parts, among them M11 Module-dinput4-0.1, M12 Module-dinput4-0.1

Commit message: EmbeddedEra libraries and template, KiCad 10
- Every symbol except the nine Hellen-One modules now comes from the EmbeddedEra library (resistors and 0R links from the generic libraries, PTC fuses, VND14NV04-E, TE 1-1376430-0, Molex 39281143, test pads, proto area, power symbols). Same-pin parts swapped in place; resistors re-placed between their old pin points with short wires. New parts live on library branch sti2004-parts.
- EmbeddedEra project template: worksheet, text variables, net classes with explicit power classes, JLCPCB design rules; template net names for USB, I2C and the K-line UART.
- Migrated all sheets and the board to KiCad 10 (10.0.7).
- tools/sch_overlap_check.py also fails on overlapping symbol bodies and on fields printed across a wire (found the stacked PTC fuses); KiCad 10 hide flags understood.

Verified: connectivity identical to the previous commit (167 nets), only the planned net renames; 0 overlaps on all 10 sheet files; ERC errors unchanged (148); pinout check 99 OK.

Co-Authored-By: Claude Opus 5.5 <noreply@anthropic.com>
Parts:
- removed R30, R31, R32, R33, R34, R44: 4.7k, hellen-one-common:R0603, symbol hellen-one-common:Res
- removed R35, R36, R37: 1k, hellen-one-common:R1206, symbol hellen-one-common:Res
- removed R45: 1k, hellen-one-common:R0603, symbol hellen-one-common:Res
- removed R51, R52, R53: 10k, hellen-one-common:R0603, symbol hellen-one-common:Res
- added R30, R31, R32, R33, R34, R44: 4.7K, EmbeddedEra_Library:R_0603_1608Metric, symbol EmbeddedEra_Resistors_0603:EE_R_0603_4.7K_1%
- added R35, R36, R37: 1K, EmbeddedEra_Library:R_1206_3216Metric, symbol EmbeddedEra_Resistors_1206:EE_R_1206_1K_1%
- added R45: 1K, EmbeddedEra_Library:R_0603_1608Metric, symbol EmbeddedEra_Resistors_0603:EE_R_0603_1K_1%
- added R51, R52, R53: 10K, EmbeddedEra_Library:R_0603_1608Metric, symbol EmbeddedEra_Resistors_0603:EE_R_0603_10K_1%
Connections:
- net +5V: now also R51.2, R52.2, R53.2
- net +5VA: now also R45.2
- net GND: now also R30.2, R31.2, R32.2, R33.2, R34.2, R35.2, R36.2, R37.2, R44.2
- net IN_AC_REQUEST: now also R31.1
- net IN_BLOWER: now also R53.1
- net IN_BRAKE_SW1: now also R34.1
- net IN_BRAKE_SW2: now also R32.1
- net IN_CLUTCH: now also R33.1
- net IN_CRUISE_MAIN: now also R35.1
- net IN_CRUISE_RESUME: now also R36.1
- net IN_CRUISE_SET: now also R37.1
- net IN_DEFOG: now also R51.1
- net IN_FUEL_LEVEL: now also R45.1
- net IN_NEUTRAL_SWITCH: now also R44.1
- net IN_SMALL_LIGHT: now also R52.1
- net IN_STARTER_SWITCH: now also R30.1
