File: Inputs.kicad_sch (KiCad schematic)
At the start: 15 parts, among them M11 Module-dinput4-0.1, M12 Module-dinput4-0.1

Commit message: Title block: TITLE is the project name (${Project_Name}) on every sheet, DESCRIPTION the sheet name
The LS/INJ sub-sheet and the root had no title at all.

Co-Authored-By: Claude Opus 5.5 <noreply@anthropic.com>
Other:
- title: Switch inputs -> ${Project_Name}
Changed lines of the file:
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@@
 	(paper "A3")
 	(title_block
-		(title "Switch inputs")
+		(title "${Project_Name}")
 		(date "2026-10-13")
 	)
