File: Mcu.kicad_sch (KiCad schematic)
At the start: 11 parts, among them J2 USB C 2.0 16P, M1 Module-mega-mcu144-0.7, P23 BOOT0, P24 SWDIO, P25 SWCLK, P26 NRST, U1 USBLC6-2SC6

Commit message: EmbeddedEra libraries and template, KiCad 10
- Every symbol except the nine Hellen-One modules now comes from the EmbeddedEra library (resistors and 0R links from the generic libraries, PTC fuses, VND14NV04-E, TE 1-1376430-0, Molex 39281143, test pads, proto area, power symbols). Same-pin parts swapped in place; resistors re-placed between their old pin points with short wires. New parts live on library branch sti2004-parts.
- EmbeddedEra project template: worksheet, text variables, net classes with explicit power classes, JLCPCB design rules; template net names for USB, I2C and the K-line UART.
- Migrated all sheets and the board to KiCad 10 (10.0.7).
- tools/sch_overlap_check.py also fails on overlapping symbol bodies and on fields printed across a wire (found the stacked PTC fuses); KiCad 10 hide flags understood.

Verified: connectivity identical to the previous commit (167 nets), only the planned net renames; 0 overlaps on all 10 sheet files; ERC errors unchanged (148); pinout check 99 OK.

Co-Authored-By: Claude Opus 5.5 <noreply@anthropic.com>
Parts:
- removed JP10: 0R, hellen-one-common:PAD-0805-PAD, symbol hellen-one-common:Jumper-Pad-Pad
- removed JP11: DNP 0R, hellen-one-common:PAD-0805-PAD, symbol hellen-one-common:Jumper-Pad-Pad
- removed P23: BOOT0, hellen-one-common:PAD-TH, symbol hellen-one-common:Pad
- removed P24: SWDIO, hellen-one-common:PAD-TH, symbol hellen-one-common:Pad
- removed P25: SWCLK, hellen-one-common:PAD-TH, symbol hellen-one-common:Pad
- removed P26: NRST, hellen-one-common:PAD-TH, symbol hellen-one-common:Pad
- removed R46, R47: 5.1k, hellen-one-common:R0603, symbol hellen-one-common:Res
- added JP10, JP11: 0, EmbeddedEra_Library:R_0805_2012Metric, symbol EmbeddedEra_Resistors_0805_5pct:EE_R_0805_0_5%
- added P23: BOOT0, EmbeddedEra_Library:TestPoint_THTPad_D2.0mm_Drill1.0mm, symbol EmbeddedEra:TestPoint_THT
- added P24: SWDIO, EmbeddedEra_Library:TestPoint_THTPad_D2.0mm_Drill1.0mm, symbol EmbeddedEra:TestPoint_THT
- added P25: SWCLK, EmbeddedEra_Library:TestPoint_THTPad_D2.0mm_Drill1.0mm, symbol EmbeddedEra:TestPoint_THT
- added P26: NRST, EmbeddedEra_Library:TestPoint_THTPad_D2.0mm_Drill1.0mm, symbol EmbeddedEra:TestPoint_THT
- added R46, R47: 5.1K, EmbeddedEra_Library:R_0603_1608Metric, symbol EmbeddedEra_Resistors_0603:EE_R_0603_5.1K_1%
- J2: footprint STI:USB_C_Receptacle_HRO_TYPE-C-31-M-12 -> EmbeddedEra_Library:USB_C_Receptacle_HRO _TYPE-C-31-M-12
- U1: footprint STI:SOT-23-6 -> EmbeddedEra_Library:SOT-23-6
Connections:
- net +3.3V: now also JP11.2
- net BOOT0: now also JP11.1, P23.1
- net GND: now also JP10.2, R46.2, R47.2
- net NRST: now also P26.1
- net SWCLK: now also P25.1
- net SWDIO: now also P24.1
- net USB_CC1: now also R46.1
- net USB_CC2: now also R47.1
- net USB_SHIELD: now also JP10.1
- net I2C_SCL renamed I2C_1_SCL
- net I2C_SDA renamed I2C_1_SDA
- net KLINE_RX renamed UART_8_RX
- net KLINE_TX renamed UART_8_TX
- net USB_DM renamed USB_D-
- net USB_DP renamed USB_D+
