File: Outputs.kicad_sch (KiCad schematic)
At the start: 11 parts, among them M2 Module-motor-driver-0.1, M9 Module-motor-driver-0.1, P10 OUT_SPARE_LS2, P12 FP_STATUS, P9 OUT_SPARE_LS1

Commit message: EmbeddedEra libraries and template, KiCad 10
- Every symbol except the nine Hellen-One modules now comes from the EmbeddedEra library (resistors and 0R links from the generic libraries, PTC fuses, VND14NV04-E, TE 1-1376430-0, Molex 39281143, test pads, proto area, power symbols). Same-pin parts swapped in place; resistors re-placed between their old pin points with short wires. New parts live on library branch sti2004-parts.
- EmbeddedEra project template: worksheet, text variables, net classes with explicit power classes, JLCPCB design rules; template net names for USB, I2C and the K-line UART.
- Migrated all sheets and the board to KiCad 10 (10.0.7).
- tools/sch_overlap_check.py also fails on overlapping symbol bodies and on fields printed across a wire (found the stacked PTC fuses); KiCad 10 hide flags understood.

Verified: connectivity identical to the previous commit (167 nets), only the planned net renames; 0 overlaps on all 10 sheet files; ERC errors unchanged (148); pinout check 99 OK.

Co-Authored-By: Claude Opus 5.5 <noreply@anthropic.com>
Parts:
- removed JP5, JP6: DNP 0R, hellen-one-common:PAD-0805-PAD, symbol hellen-one-common:Jumper-Pad-Pad
- removed P10: OUT_SPARE_LS2, hellen-one-common:PAD-TH, symbol hellen-one-common:Pad
- removed P12: FP_STATUS, hellen-one-common:PAD-TH, symbol hellen-one-common:Pad
- removed P9: OUT_SPARE_LS1, hellen-one-common:PAD-TH, symbol hellen-one-common:Pad
- removed R38: 2.2k, hellen-one-common:R0805, symbol hellen-one-common:Res
- removed R39: 100, hellen-one-common:R0603, symbol hellen-one-common:Res
- removed R40: 1k, hellen-one-common:R0603, symbol hellen-one-common:Res
- removed R41: 10k, hellen-one-common:R0603, symbol hellen-one-common:Res
- added JP5, JP6: 0, EmbeddedEra_Library:R_0805_2012Metric, symbol EmbeddedEra_Resistors_0805_5pct:EE_R_0805_0_5%
- added P10: OUT_SPARE_LS2, EmbeddedEra_Library:TestPoint_THTPad_D2.0mm_Drill1.0mm, symbol EmbeddedEra:TestPoint_THT
- added P12: FP_STATUS, EmbeddedEra_Library:TestPoint_THTPad_D2.0mm_Drill1.0mm, symbol EmbeddedEra:TestPoint_THT
- added P9: OUT_SPARE_LS1, EmbeddedEra_Library:TestPoint_THTPad_D2.0mm_Drill1.0mm, symbol EmbeddedEra:TestPoint_THT
- added R38: 2.2k, EmbeddedEra_Library:R_0805_2012Metric, symbol EmbeddedEra_Resistors_0805_5pct:EE_R_0805_2.2k_5%
- added R39: 100, EmbeddedEra_Library:R_0603_1608Metric, symbol EmbeddedEra_Resistors_0603:EE_R_0603_100_1%
- added R40: 1K, EmbeddedEra_Library:R_0603_1608Metric, symbol EmbeddedEra_Resistors_0603:EE_R_0603_1K_1%
- added R41: 10K, EmbeddedEra_Library:R_0603_1608Metric, symbol EmbeddedEra_Resistors_0603:EE_R_0603_10K_1%
Connections:
- net +12V_RAW: now also R38.2
- net +5V: now also R40.2
- net EVAP_A12: now also JP5.2
- net EVAP_A13: now also JP6.2
- net FP_CMD: now also R39.1
- net FP_STATUS: now also P12.1
- net FUEL_PUMP_SIGNAL1: now also R39.2, R40.1, R41.1
- net GND: now also R41.2
- net OUT_SPARE_LS1: now also JP5.1, P9.1
- net OUT_SPARE_LS2: now also JP6.1, P10.1
- net OUT_TACH: now also R38.1
