File: Aux.kicad_sch (KiCad schematic)
At the start: 23 parts, among them J3 MiniFitJr_2x07_AUX, P11 CHARGE_A22, P14 SPARE_IGN6, P15 SPARE_IGN7, P16 SPARE_IGN8, P17 I2C_SCL, P18 I2C_SDA, P19 +5VA, P20 +3.3V, P21 +12V_RAW, P22 GND, P27 SPARE_PWM3, P28 SPARE_RES2, P29 AUX_IN1, P30 AUX_IN2, P31 AUX_IN3

Commit message: EmbeddedEra libraries and template, KiCad 10
- Every symbol except the nine Hellen-One modules now comes from the EmbeddedEra library (resistors and 0R links from the generic libraries, PTC fuses, VND14NV04-E, TE 1-1376430-0, Molex 39281143, test pads, proto area, power symbols). Same-pin parts swapped in place; resistors re-placed between their old pin points with short wires. New parts live on library branch sti2004-parts.
- EmbeddedEra project template: worksheet, text variables, net classes with explicit power classes, JLCPCB design rules; template net names for USB, I2C and the K-line UART.
- Migrated all sheets and the board to KiCad 10 (10.0.7).
- tools/sch_overlap_check.py also fails on overlapping symbol bodies and on fields printed across a wire (found the stacked PTC fuses); KiCad 10 hide flags understood.

Verified: connectivity identical to the previous commit (167 nets), only the planned net renames; 0 overlaps on all 10 sheet files; ERC errors unchanged (148); pinout check 99 OK.

Co-Authored-By: Claude Opus 5.5 <noreply@anthropic.com>
Parts:
- removed F6: nSMD050-24V, hellen-one-common:PAD-1206-PAD, symbol hellen-one-common:Fuse-Pad-Pad
- removed F7: nSMD005, hellen-one-common:PAD-1206-PAD, symbol hellen-one-common:Fuse-Pad-Pad
- removed G1: PROTO_AREA, hellen-one-common:PROTO_AREA, symbol hellen-one-common:PROTO_AREA
- removed J3: MiniFitJr_2x07_AUX, STI:Molex_Mini-Fit_Jr_5566-14A_2x07_P4.20mm_Vertical, symbol Connector_Generic:Conn_02x07_Odd_Even
- removed JP7: DNP 0R, hellen-one-common:PAD-0805-PAD, symbol hellen-one-common:Jumper-Pad-Pad
- removed P11: CHARGE_A22, hellen-one-common:PAD-TH, symbol hellen-one-common:Pad
- removed P14: SPARE_IGN6, hellen-one-common:PAD-TH, symbol hellen-one-common:Pad
- removed P15: SPARE_IGN7, hellen-one-common:PAD-TH, symbol hellen-one-common:Pad
- removed P16: SPARE_IGN8, hellen-one-common:PAD-TH, symbol hellen-one-common:Pad
- removed P17: I2C_SCL, hellen-one-common:PAD-TH, symbol hellen-one-common:Pad
- removed P18: I2C_SDA, hellen-one-common:PAD-TH, symbol hellen-one-common:Pad
- removed P19: +5VA, hellen-one-common:PAD-TH, symbol hellen-one-common:Pad
- removed P20: +3.3V, hellen-one-common:PAD-TH, symbol hellen-one-common:Pad
- removed P21: +12V_RAW, hellen-one-common:PAD-TH, symbol hellen-one-common:Pad
- removed P22: GND, hellen-one-common:PAD-TH, symbol hellen-one-common:Pad
- removed P27: SPARE_PWM3, hellen-one-common:PAD-TH, symbol hellen-one-common:Pad
- removed P28: SPARE_RES2, hellen-one-common:PAD-TH, symbol hellen-one-common:Pad
- removed P29: AUX_IN1, hellen-one-common:PAD-TH, symbol hellen-one-common:Pad
- removed P30: AUX_IN2, hellen-one-common:PAD-TH, symbol hellen-one-common:Pad
- removed P31: AUX_IN3, hellen-one-common:PAD-TH, symbol hellen-one-common:Pad
- removed R48, R49, R50: 4.7k, hellen-one-common:R0603, symbol hellen-one-common:Res
- added F6: nSMD050-24V, EmbeddedEra_Library:Fuse_1206_3216Metric, symbol EmbeddedEra:nSMD050-24V
- added F7: JK-nSMD005, EmbeddedEra_Library:Fuse_1206_3216Metric, symbol EmbeddedEra:JK-nSMD005
- added G1: PROTO_AREA, EmbeddedEra_Library:PROTO_AREA_3x5_P2.54mm, symbol EmbeddedEra:PROTO_AREA
- added J3: Molex_39281143, EmbeddedEra_Library:Molex_Mini-Fit_Jr_5566-14A_2x07_P4.20mm_Vertical, symbol EmbeddedEra:Molex_39281143
- added JP7: 0, EmbeddedEra_Library:R_0805_2012Metric, symbol EmbeddedEra_Resistors_0805_5pct:EE_R_0805_0_5%
- added P11: CHARGE_A22, EmbeddedEra_Library:TestPoint_THTPad_D2.0mm_Drill1.0mm, symbol EmbeddedEra:TestPoint_THT
- added P14: SPARE_IGN6, EmbeddedEra_Library:TestPoint_THTPad_D2.0mm_Drill1.0mm, symbol EmbeddedEra:TestPoint_THT
- added P15: SPARE_IGN7, EmbeddedEra_Library:TestPoint_THTPad_D2.0mm_Drill1.0mm, symbol EmbeddedEra:TestPoint_THT
- added P16: SPARE_IGN8, EmbeddedEra_Library:TestPoint_THTPad_D2.0mm_Drill1.0mm, symbol EmbeddedEra:TestPoint_THT
- added P17: I2C_1_SCL, EmbeddedEra_Library:TestPoint_THTPad_D2.0mm_Drill1.0mm, symbol EmbeddedEra:TestPoint_THT
- added P18: I2C_1_SDA, EmbeddedEra_Library:TestPoint_THTPad_D2.0mm_Drill1.0mm, symbol EmbeddedEra:TestPoint_THT
- added P19: +5VA, EmbeddedEra_Library:TestPoint_THTPad_D2.0mm_Drill1.0mm, symbol EmbeddedEra:TestPoint_THT
- added P20: +3.3V, EmbeddedEra_Library:TestPoint_THTPad_D2.0mm_Drill1.0mm, symbol EmbeddedEra:TestPoint_THT
- added P21: +12V_RAW, EmbeddedEra_Library:TestPoint_THTPad_D2.0mm_Drill1.0mm, symbol EmbeddedEra:TestPoint_THT
- added P22: GND, EmbeddedEra_Library:TestPoint_THTPad_D2.0mm_Drill1.0mm, symbol EmbeddedEra:TestPoint_THT
- added P27: SPARE_PWM3, EmbeddedEra_Library:TestPoint_THTPad_D2.0mm_Drill1.0mm, symbol EmbeddedEra:TestPoint_THT
- added P28: SPARE_RES2, EmbeddedEra_Library:TestPoint_THTPad_D2.0mm_Drill1.0mm, symbol EmbeddedEra:TestPoint_THT
- added P29: AUX_IN1, EmbeddedEra_Library:TestPoint_THTPad_D2.0mm_Drill1.0mm, symbol EmbeddedEra:TestPoint_THT
- added P30: AUX_IN2, EmbeddedEra_Library:TestPoint_THTPad_D2.0mm_Drill1.0mm, symbol EmbeddedEra:TestPoint_THT
- added P31: AUX_IN3, EmbeddedEra_Library:TestPoint_THTPad_D2.0mm_Drill1.0mm, symbol EmbeddedEra:TestPoint_THT
- added R48, R49, R50: 4.7K, EmbeddedEra_Library:R_0603_1608Metric, symbol EmbeddedEra_Resistors_0603:EE_R_0603_4.7K_1%
Connections:
- net +12V_RAW: now also F6.1, P21.1
- net +3.3V: now also P20.1
- net +5VA: now also P19.1
- net +5VAS: now also F7.1
- net AUX_12V: now also F6.2, J3.1 (Pin_1)
- net AUX_5V: now also F7.2, J3.3 (Pin_3)
- net AUX_AN2: now also J3.9 (Pin_9), JP7.2
- net AUX_IN1: now also J3.5 (Pin_5), P29.1, R48.1
- net AUX_IN2: now also J3.6 (Pin_6), P30.1, R49.1
- net AUX_IN3: now also J3.7 (Pin_7), P31.1, R50.1
- net CAN_H: now also J3.12 (Pin_12)
- net CAN_L: now also J3.13 (Pin_13)
- net CHARGE_A22: now also P11.1
- net FP_STATUS: now also JP7.1
- net GND: now also J3.14 (Pin_14), J3.2 (Pin_2), P22.1, R48.2, R49.2, R50.2
- net GND_SENSOR: now also J3.4 (Pin_4)
- net OUT_SPARE_LS1: now also J3.10 (Pin_10)
- net OUT_SPARE_LS2: now also J3.11 (Pin_11)
- net SPARE_IGN6: now also P14.1
- net SPARE_IGN7: now also P15.1
- net SPARE_IGN8: now also P16.1
- net SPARE_PWM3: now also P27.1
- net SPARE_RES2: now also J3.8 (Pin_8), P28.1
- new net I2C_1_SCL: P17.1
- new net I2C_1_SDA: P18.1
Other:
- note added: "D: B137"

Commit message: Remove unused M7 knock module and a stray plug note; checker models KiCad's field-justify flip
- M7 (second knock module) had no pin connected; the STI has one knock sensor (C25) on M13.
- 'D: B137' free text (rev-a leftover) duplicated J1's own plug label and sat on the Aux sheet.
- sch_overlap_check: KiCad draws a field's left/right justification mirrored for some
  angle/rotation/mirror combinations (measured from kicad-cli 10 PDF output); the checker now
  boxes those fields where KiCad draws them.

Co-Authored-By: Claude Opus 5.5 <noreply@anthropic.com>
Other:
- note removed: "D: B137"
Changed lines of the file:
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@@
-		)
-	)
-	(text "D: B137"
-		(exclude_from_sim no)
-		(at 99.314 93.726 0)
-		(effects
-			(font
-				(size 1.27 1.27)
-			)
 		)
 	)
