File: INJ4.kicad_sch (KiCad schematic)
At the start: 8 parts, among them Q1 VND14NV04-E, Q2 VND14NV04-E, Q3 VND14NV04-E, Q4 VND14NV04-E

Commit message: Low-side drivers Q1-Q20: VND14NV04-E (obsolete) -> onsemi NCV8401BDTRKG
Same DPAK pinout and TO-252-2 footprint; protected (active clamp, current limit, thermal
shutdown), AEC-Q101, about 28 mOhm at 5 V. Netlist unchanged, 0 overlaps. Schematic PDF
regenerated.

Co-Authored-By: Claude Opus 5.5 <noreply@anthropic.com>
Parts:
- Q1, Q2, Q3, Q4: value VND14NV04-E -> NCV8401BDTRKG; symbol EmbeddedEra:VND14NV04-E -> EmbeddedEra:NCV8401BDTRKG; LCSC C155647 -> (none); Manufacturer STMicroelectronics -> onsemi; Manufacturer Part Number VND14NV04-E -> NCV8401BDTRKG
Changed lines of the file:
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@@
 	)
 	(symbol
-		(lib_id "EmbeddedEra:VND14NV04-E")
+		(lib_id "EmbeddedEra:NCV8401BDTRKG")
 		(at 149.86 123.19 0)
 		(mirror y)
@@
 			)
 		)
-		(property "Value" "VND14NV04-E"
+		(property "Value" "NCV8401BDTRKG"
 			(at 146.05 124.46 0)
 			(show_name no)
@@
 			)
 		)
-		(property "Datasheet" "https://www.st.com/resource/en/datasheet/vnd14nv04-e.pdf"
+		(property "Datasheet" "https://www.onsemi.com/pdf/datasheet/ncv8401-d.pdf"
 			(at 149.86 123.19 0)
 			(hide yes)
@@
 			)
 		)
-		(property "Description" "VND14NV04-E OMNIFET II LOW SIDE POWER SWITCH 40V 14MOHM DPAK"
+		(property "Description" "NCV8401BDTRKG SELF-PROTECTED LOW SIDE DRIVER 42V 33A 23MOHM DPAK"
 			(at 149.86 123.19 0)
 			(hide yes)
@@
 			)
 		)
-		(property "LCSC" "C155647"
+		(property "LCSC" ""
 			(at 149.86 123.19 0)
 			(hide yes)
@@
 			)
 		)
-		(property "Manufacturer" "STMicroelectronics"
+		(property "Manufacturer" "onsemi"
 			(at 149.86 123.19 0)
 			(hide yes)
@@
 			)
 		)
-		(property "Manufacturer Part Number" "VND14NV04-E"
+		(property "Manufacturer Part Number" "NCV8401BDTRKG"
 			(at 149.86 123.19 0)
 			(hide yes)
@@
 	)
 	(symbol
-		(lib_id "EmbeddedEra:VND14NV04-E")
+		(lib_id "EmbeddedEra:NCV8401BDTRKG")
 		(at 149.86 58.42 0)
 		(mirror y)
@@
 			)
 		)
-		(property "Value" "VND14NV04-E"
+		(property "Value" "NCV8401BDTRKG"
 			(at 146.05 59.69 0)
 			(show_name no)
@@
 			)
 		)
-		(property "Datasheet" "https://www.st.com/resource/en/datasheet/vnd14nv04-e.pdf"
+		(property "Datasheet" "https://www.onsemi.com/pdf/datasheet/ncv8401-d.pdf"
 			(at 149.86 58.42 0)
 			(hide yes)
@@
 			)
 		)
-		(property "Description" "VND14NV04-E OMNIFET II LOW SIDE POWER SWITCH 40V 14MOHM DPAK"
+		(property "Description" "NCV8401BDTRKG SELF-PROTECTED LOW SIDE DRIVER 42V 33A 23MOHM DPAK"
 			(at 149.86 58.42 0)
 			(hide yes)
@@
 			)
 		)
-		(property "LCSC" "C155647"
+		(property "LCSC" ""
 			(at 149.86 58.42 0)
 			(hide yes)
@@
 			)
 		)
-		(property "Manufacturer" "STMicroelectronics"
+		(property "Manufacturer" "onsemi"
 			(at 149.86 58.42 0)
 			(hide yes)
@@
 			)
 		)
-		(property "Manufacturer Part Number" "VND14NV04-E"
+		(property "Manufacturer Part Number" "NCV8401BDTRKG"
 			(at 149.86 58.42 0)
 			(hide yes)
@@
 	)
 	(symbol
-		(lib_id "EmbeddedEra:VND14NV04-E")
+		(lib_id "EmbeddedEra:NCV8401BDTRKG")
 		(at 149.86 80.01 0)
 		(mirror y)
@@
 			)
 		)
-		(property "Value" "VND14NV04-E"
+		(property "Value" "NCV8401BDTRKG"
 			(at 146.05 81.28 0)
 			(show_name no)
@@
 			)
 		)
-		(property "Datasheet" "https://www.st.com/resource/en/datasheet/vnd14nv04-e.pdf"
+		(property "Datasheet" "https://www.onsemi.com/pdf/datasheet/ncv8401-d.pdf"
 			(at 149.86 80.01 0)
 			(hide yes)
@@
 			)
 		)
-		(property "Description" "VND14NV04-E OMNIFET II LOW SIDE POWER SWITCH 40V 14MOHM DPAK"
+		(property "Description" "NCV8401BDTRKG SELF-PROTECTED LOW SIDE DRIVER 42V 33A 23MOHM DPAK"
 			(at 149.86 80.01 0)
 			(hide yes)
@@
 			)
 		)
-		(property "LCSC" "C155647"
+		(property "LCSC" ""
 			(at 149.86 80.01 0)
 			(hide yes)
@@
 			)
 		)
-		(property "Manufacturer" "STMicroelectronics"
+		(property "Manufacturer" "onsemi"
 			(at 149.86 80.01 0)
 			(hide yes)
@@
 			)
 		)
-		(property "Manufacturer Part Number" "VND14NV04-E"
+		(property "Manufacturer Part Number" "NCV8401BDTRKG"
 			(at 149.86 80.01 0)
 			(hide yes)
@@
 	)
 	(symbol
-		(lib_id "EmbeddedEra:VND14NV04-E")
+		(lib_id "EmbeddedEra:NCV8401BDTRKG")
 		(at 149.86 101.6 0)
 		(mirror y)
@@
 			)
 		)
-		(property "Value" "VND14NV04-E"
+		(property "Value" "NCV8401BDTRKG"
 			(at 146.05 102.87 0)
 			(show_name no)
@@
 			)
 		)
-		(property "Datasheet" "https://www.st.com/resource/en/datasheet/vnd14nv04-e.pdf"
+		(property "Datasheet" "https://www.onsemi.com/pdf/datasheet/ncv8401-d.pdf"
 			(at 149.86 101.6 0)
 			(hide yes)
@@
 			)
 		)
-		(property "Description" "VND14NV04-E OMNIFET II LOW SIDE POWER SWITCH 40V 14MOHM DPAK"
+		(property "Description" "NCV8401BDTRKG SELF-PROTECTED LOW SIDE DRIVER 42V 33A 23MOHM DPAK"
 			(at 149.86 101.6 0)
 			(hide yes)
@@
 			)
 		)
-		(property "LCSC" "C155647"
+		(property "LCSC" ""
 			(at 149.86 101.6 0)
 			(hide yes)
@@
 			)
 		)
-		(property "Manufacturer" "STMicroelectronics"
+		(property "Manufacturer" "onsemi"
 			(at 149.86 101.6 0)
 			(hide yes)
@@
 			)
 		)
-		(property "Manufacturer Part Number" "VND14NV04-E"
+		(property "Manufacturer Part Number" "NCV8401BDTRKG"
 			(at 149.86 101.6 0)
 			(hide yes)

Commit message: Title block: TITLE is the project name (${Project_Name}) on every sheet, DESCRIPTION the sheet name
The LS/INJ sub-sheet and the root had no title at all.

Co-Authored-By: Claude Opus 5.5 <noreply@anthropic.com>
Other:
- title: (none) -> ${Project_Name}
Changed lines of the file:
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@@
 	(generator_version "10.0")
 	(paper "A4")
+	(title_block
+		(title "${Project_Name}")
+		(date "2026-10-13")
+	)
 	(junction
 		(at 167.64 123.19)
