File: Power.kicad_sch (KiCad schematic)
At the start: 4 parts, among them M14 Module-power_12and5V-0.3, M8 Module-power_12and5V-0.3, P32 PG_5VP_APS

Commit message: U1 is the library USBLC6-2SC6 (EE-C-0146); J2 part numbers; test pads and proto area out of the BOM
- U1 used the USBLC6-2P6 (SOT-666) symbol with a hand-changed footprint; now EmbeddedEra:USBLC6-2SC6.
- J2 instance had no Manufacturer/MPN although the library has them.
- P1-P32 and G1 are pads, nothing is bought (SOP-008 step 18): in_bom no, as in the library.

Co-Authored-By: Claude Opus 5.5 <noreply@anthropic.com>
Parts:
- P32: now left out of the parts list
Changed lines of the file:
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@@
 		(body_style 1)
 		(exclude_from_sim no)
-		(in_bom yes)
+		(in_bom no)
 		(on_board yes)
 		(in_pos_files yes)

Commit message: Title block: TITLE is the project name (${Project_Name}) on every sheet, DESCRIPTION the sheet name
The LS/INJ sub-sheet and the root had no title at all.

Co-Authored-By: Claude Opus 5.5 <noreply@anthropic.com>
Other:
- title: Power -> ${Project_Name}
Changed lines of the file:
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@@
 	(paper "A3")
 	(title_block
-		(title "Power")
+		(title "${Project_Name}")
 		(date "2026-10-13")
 	)
