File: Sensors.kicad_sch (KiCad schematic)
At the start: 6 parts, among them M13 Module-knock-0.2, M5 Module-vr-discrete-0.5

Commit message: Title block: TITLE is the project name (${Project_Name}) on every sheet, DESCRIPTION the sheet name
The LS/INJ sub-sheet and the root had no title at all.

Co-Authored-By: Claude Opus 5.5 <noreply@anthropic.com>
Other:
- title: Sensors -> ${Project_Name}
Changed lines of the file:
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@@
 	(paper "A3")
 	(title_block
-		(title "Sensors")
+		(title "${Project_Name}")
 		(date "2026-10-13")
 	)
