File: LS_MIX.kicad_sch (KiCad schematic)
At the start: 8 parts, among them Q1 NCV8401BDTRKG, Q2 NCV8401BDTRKG, Q3 NCV8401BDTRKG, Q4 NCV8401BDTRKG

Commit message: Low-side drivers as on the newest rusEFI boards: 10 x VNLD5160 dual SO-8 + 1 NCV8401B DPAK for the rear O2 heater
rusEFI uaefi-f, hellen-112-17 and hellen154hyundai-e use VNLD5090/VNLD5160 for general outputs and
keep one DPAK for the heaviest load; our Hellen modules already carry their other ICs. Every output
keeps its J1 and MCU pin (netlist checked); U19B parked as a spare. PCB re-placed: DRC 0 errors.

Co-Authored-By: Claude Opus 5.5 <noreply@anthropic.com>
Parts:
- added unit 2 of U2
- U1: renamed from Q1; value NCV8401BDTRKG -> VNLD5160TR-E; footprint EmbeddedEra_Library:TO-252-2 -> EmbeddedEra_Library:SOIC-8_3.9x4.9mm_P1.27mm; symbol EmbeddedEra:NCV8401BDTRKG -> EmbeddedEra:VNLD5160TR-E; LCSC (none) -> C377942; Manufacturer onsemi -> STMicroelectronics; Manufacturer Part Number NCV8401BDTRKG -> VNLD5160TR-E
- U1: renamed from Q2; value NCV8401BDTRKG -> VNLD5160TR-E; footprint EmbeddedEra_Library:TO-252-2 -> EmbeddedEra_Library:SOIC-8_3.9x4.9mm_P1.27mm; symbol EmbeddedEra:NCV8401BDTRKG -> EmbeddedEra:VNLD5160TR-E; LCSC (none) -> C377942; Manufacturer onsemi -> STMicroelectronics; Manufacturer Part Number NCV8401BDTRKG -> VNLD5160TR-E
- U2: renamed from Q3; value NCV8401BDTRKG -> VNLD5160TR-E; footprint EmbeddedEra_Library:TO-252-2 -> EmbeddedEra_Library:SOIC-8_3.9x4.9mm_P1.27mm; symbol EmbeddedEra:NCV8401BDTRKG -> EmbeddedEra:VNLD5160TR-E; LCSC (none) -> C377942; Manufacturer onsemi -> STMicroelectronics; Manufacturer Part Number NCV8401BDTRKG -> VNLD5160TR-E
Connections:
- net GND: now also U1.5 (S), U1.7 (S), U2.7 (S), U2.5 (S); no longer U1.3 (S), U1.3 (S), U2.3 (S)
- net IN2: now also U1.3 (IN); no longer U1.1 (IN)
- net OUT1: now also U1.8 (D); no longer U1.2 (D)
- net OUT2: now also U1.6 (D); no longer U1.2 (D)
- net OUT3: now also U2.8 (D); no longer U2.2 (D)
- no-connect marks 0 -> 6
Other:
- note added: "U19 channel 2: unused spare (input and drain open, as the datasheet allows)."
