File: LS_VNLD.kicad_sch (KiCad schematic)
At the start: 8 parts, among them Q1 ZXMS6004FFTA, Q2 ZXMS6004FFTA, Q3 ZXMS6004FFTA, Q4 ZXMS6004FFTA

Commit message: Low-side drivers as on the newest rusEFI boards: 10 x VNLD5160 dual SO-8 + 1 NCV8401B DPAK for the rear O2 heater
rusEFI uaefi-f, hellen-112-17 and hellen154hyundai-e use VNLD5090/VNLD5160 for general outputs and
keep one DPAK for the heaviest load; our Hellen modules already carry their other ICs. Every output
keeps its J1 and MCU pin (netlist checked); U19B parked as a spare. PCB re-placed: DRC 0 errors.

Co-Authored-By: Claude Opus 5.5 <noreply@anthropic.com>
Parts:
- U1: renamed from Q1; value ZXMS6004FFTA -> VNLD5160TR-E; footprint EmbeddedEra_Library:SOT-23F_Diodes -> EmbeddedEra_Library:SOIC-8_3.9x4.9mm_P1.27mm; symbol EmbeddedEra:ZXMS6004FFTA -> EmbeddedEra:VNLD5160TR-E; LCSC C95063 -> C377942; Manufacturer Diodes Incorporated -> STMicroelectronics; Manufacturer Part Number ZXMS6004FFTA -> VNLD5160TR-E
- U1: renamed from Q2; value ZXMS6004FFTA -> VNLD5160TR-E; footprint EmbeddedEra_Library:SOT-23F_Diodes -> EmbeddedEra_Library:SOIC-8_3.9x4.9mm_P1.27mm; symbol EmbeddedEra:ZXMS6004FFTA -> EmbeddedEra:VNLD5160TR-E; LCSC C95063 -> C377942; Manufacturer Diodes Incorporated -> STMicroelectronics; Manufacturer Part Number ZXMS6004FFTA -> VNLD5160TR-E
- U2: renamed from Q4; value ZXMS6004FFTA -> VNLD5160TR-E; footprint EmbeddedEra_Library:SOT-23F_Diodes -> EmbeddedEra_Library:SOIC-8_3.9x4.9mm_P1.27mm; symbol EmbeddedEra:ZXMS6004FFTA -> EmbeddedEra:VNLD5160TR-E; LCSC C95063 -> C377942; Manufacturer Diodes Incorporated -> STMicroelectronics; Manufacturer Part Number ZXMS6004FFTA -> VNLD5160TR-E
- U2: renamed from Q3; value ZXMS6004FFTA -> VNLD5160TR-E; footprint EmbeddedEra_Library:SOT-23F_Diodes -> EmbeddedEra_Library:SOIC-8_3.9x4.9mm_P1.27mm; symbol EmbeddedEra:ZXMS6004FFTA -> EmbeddedEra:VNLD5160TR-E; LCSC C95063 -> C377942; Manufacturer Diodes Incorporated -> STMicroelectronics; Manufacturer Part Number ZXMS6004FFTA -> VNLD5160TR-E
Connections:
- net GND: now also U1.5 (S), U1.7 (S), U2.5 (S), U2.7 (S); no longer U1.2 (S), U1.2 (S), U2.2 (S), U2.2 (S)
- net IN2: now also U1.3 (IN); no longer U1.1 (IN)
- net IN4: now also U2.3 (IN); no longer U2.1 (IN)
- net OUT1: now also U1.8 (D); no longer U1.3 (D)
- net OUT2: now also U1.6 (D); no longer U1.3 (D)
- net OUT3: now also U2.8 (D); no longer U2.3 (D)
- net OUT4: now also U2.6 (D); no longer U2.3 (D)
- no-connect marks 0 -> 4
